File: EEE3088/Power_kicad_sch.kicad_sch (KiCad schematic)
At the start: 22 parts, among them Q1 LBSS84LT1G, U1 TP4056, U2 HT7533-1

Commit message: power updates
Parts:
- removed Q1: LBSS84LT1G, SOT96P237X111-3N, symbol LBSS84LT1G:LBSS84LT1G
- added P-Mos: AO3401A, SOT95P280X125-3N, symbol AO3401A:AO3401A
Connections:
- net V-pos: now also P-Mos.2
- net at D1.A, R5.2: now also P-Mos.1
- net at BT1.P: now also P-Mos.3
Changed lines of the file:
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@@
-    )
-  )
-  (symbol (lib_id "LBSS84LT1G:LBSS84LT1G") (at 38.1 116.84 90) (unit 1)
-    (in_bom yes) (on_board yes) (dnp no) (fields_autoplaced)
-    (property "Reference" "Q1" (at 35.56 102.87 90)
-      (effects (font (size 1.27 1.27)))
-    )
-    (property "Value" "LBSS84LT1G" (at 35.56 105.41 90)
-      (effects (font (size 1.27 1.27)))
-    )
-    (property "Footprint" "SOT96P237X111-3N" (at 39.37 105.41 0)
-      (effects (font (size 1.27 1.27)) (justify left) hide)
-    )
-    (property "Datasheet" "https://datasheet.lcsc.com/lcsc/1811031711_LRC-LBSS84LT1G_C8492.pdf" (at 41.91 105.41 0)
-      (effects (font (size 1.27 1.27)) (justify left) hide)
-    )
-    (property "Description" "P-MOSFET" (at 44.45 105.41 0)
-      (effects (font (size 1.27 1.27)) (justify left) hide)
-    )
-    (property "Height" "1.11" (at 46.99 105.41 0)
-      (effects (font (size 1.27 1.27)) (justify left) hide)
-    )
-    (property "Manufacturer_Name" "onsemi" (at 49.53 105.41 0)
-      (effects (font (size 1.27 1.27)) (justify left) hide)
-    )
-    (property "Manufacturer_Part_Number" "LBSS84LT1G" (at 52.07 105.41 0)
-      (effects (font (size 1.27 1.27)) (justify left) hide)
-    )
-    (property "Mouser Part Number" "N/A" (at 54.61 105.41 0)
-      (effects (font (size 1.27 1.27)) (justify left) hide)
-    )
-    (property "Mouser Price/Stock" "https://www.mouser.co.uk/ProductDetail/onsemi/LBSS84LT1G?qs=k4J6HQLAy0oy6qnSSn%252B1%252BA%3D%3D" (at 57.15 105.41 0)
-      (effects (font (size 1.27 1.27)) (justify left) hide)
-    )
-    (property "Arrow Part Number" "" (at 59.69 105.41 0)
-      (effects (font (size 1.27 1.27)) (justify left) hide)
-    )
-    (property "Arrow Price/Stock" "" (at 62.23 105.41 0)
-      (effects (font (size 1.27 1.27)) (justify left) hide)
-    )
-    (property "Price" "0.0242" (at 38.1 116.84 0)
-      (effects (font (size 1.27 1.27)) hide)
-    )
-    (property "Basic" "" (at 38.1 116.84 0)
-      (effects (font (size 1.27 1.27)) hide)
-    )
-    (property "Extended" "0" (at 38.1 116.84 0)
-      (effects (font (size 1.27 1.27)) hide)
-    )
-    (pin "1")
-    (pin "2")
-    (pin "3")
-    (instances
-      (project "Power_kicad_sch"
-        (path "/02e53f89-135a-4459-982b-e3c28e008824"
-          (reference "Q1") (unit 1)
-        )
-      )
-      (project "EEE3088"
-        (path "/83bdd5e1-981a-4ca1-9a2f-70dea9f00850/1213f935-6f8d-4a20-9c2e-6b5e9a834fe6"
-          (reference "P-Mos1") (unit 1)
-        )
-      )
     )
   )
@@
         )
       )
+    )
+  )
+  (symbol (lib_id "AO3401A:AO3401A") (at 38.1 116.84 90) (unit 1)
+    (in_bom yes) (on_board yes) (dnp no) (fields_autoplaced)
+    (property "Reference" "P-Mos" (at 35.56 102.87 90)
+      (effects (font (size 1.27 1.27)))
+    )
+    (property "Value" "AO3401A" (at 35.56 105.41 90)
+      (effects (font (size 1.27 1.27)))
+    )
+    (property "Footprint" "SOT95P280X125-3N" (at 39.37 105.41 0)
+      (effects (font (size 1.27 1.27)) (justify left) hide)
+    )
+    (property "Datasheet" "https://datasheet.lcsc.com/lcsc/1810171817_Alpha---Omega-Semicon-AO3401A_C15127.pdf" (at 41.91 105.41 0)
+      (effects (font (size 1.27 1.27)) (justify left) hide)
+    )
+    (property "Description" "30V P-Channel MOSFET" (at 44.45 105.41 0)
+      (effects (font (size 1.27 1.27)) (justify left) hide)
+    )
+    (property "Height" "1.25" (at 46.99 105.41 0)
+      (effects (font (size 1.27 1.27)) (justify left) hide)
+    )
+    (property "Manufacturer_Name" "Alpha & Omega Semiconductors" (at 49.53 105.41 0)
+      (effects (font (size 1.27 1.27)) (justify left) hide)
+    )
+    (property "Manufacturer_Part_Number" "AO3401A" (at 52.07 105.41 0)
+      (effects (font (size 1.27 1.27)) (justify left) hide)
+    )
+    (property "Mouser Part Number" "" (at 54.61 105.41 0)
+      (effects (font (size 1.27 1.27)) (justify left) hide)
+    )
+    (property "Mouser Price/Stock" "" (at 57.15 105.41 0)
+      (effects (font (size 1.27 1.27)) (justify left) hide)
+    )
+    (property "Arrow Part Number" "AO3401A" (at 59.69 105.41 0)
+      (effects (font (size 1.27 1.27)) (justify left) hide)
+    )
+    (property "Arrow Price/Stock" "https://www.arrow.com/en/products/ao3401a/alpha-and-omega-semiconductor?region=nac" (at 62.23 105.41 0)
+      (effects (font (size 1.27 1.27)) (justify left) hide)
+    )
+    (property "Extended" "0" (at 38.1 116.84 0)
+      (effects (font (size 1.27 1.27)) hide)
+    )
+    (property "Price" "0.0797" (at 38.1 116.84 0)
+      (effects (font (size 1.27 1.27)) hide)
+    )
+    (pin "1")
+    (pin "2")
+    (pin "3")
+    (instances
+      (project "EEE3088"
+        (path "/83bdd5e1-981a-4ca1-9a2f-70dea9f00850/1213f935-6f8d-4a20-9c2e-6b5e9a834fe6"
+          (reference "P-Mos") (unit 1)
+        )
+      )

Commit message: power edit
Parts:
- added R10, R4, R6, R8, R9: 0, RESC1005X40N, symbol 0402WGF0000TCE:0402WGF0000TCE
- renumbered P-Mos to P-Mos1, R3 to R7, TP9 to TP1, TP8 to TP2, TP10 to TP3, TP11 to TP4, TP12 to TP5
Connections:
- net +3.3V: now also R9.2; no longer TP5.1, U2.3 (VO)
- net 3.3-back: now also R10.2; no longer TP4.1, Voltage-Regulator-1.3 (VO)
- net V-Reg: now also R8.2; no longer N-Mos1.2, R7.1, TP3.1
- net V-pos: now also R4.2; no longer D1.C, P-Mos1.2, TP1.1
- net Vbat: now also R6.2; no longer C2.1, TP2.1, U1.5 (BAT)
- new net: N-Mos1.2, R7.1, R8.1, TP3.1
- new net: R10.1, TP4.1, Voltage-Regulator-1.3 (VO)
- new net: R9.1, TP5.1, U2.3 (VO)
- new net: C2.1, R6.1, TP2.1, U1.5 (BAT)
- new net: D1.C, P-Mos1.2, R4.1, TP1.1
Other:
- moved on the sheet: N-Mos1, Op-Amp1, R7, TP3, TP4, TP5, U2, Voltage-Regulator-1

Commit message: BOM attempt
Parts:
- BT1: Manufacturer_Part_Number (none) -> -
- D1: Extended (none) -> -; Manufacturer_Part_Number (none) -> -; Price (none) -> -
- R10, R4, R6, R8, R9: Extended (none) -> 0; Price (none) -> 0.0035
- TP1, TP2, TP3, TP4, TP5: Extended (none) -> 0; Manufacturer_Part_Number (none) -> 0; Price (none) -> 0
Changed lines of the file:
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@@
       (effects (font (size 1.27 1.27)) (justify left) hide)
     )
-    (property "Description" "Thick Film Resistors - SMD 0402 1/16W 1% 0R T/R-10000" (at 231.775 135.89 0)
+    (property "Description" "0 Resistor - 0402" (at 231.775 135.89 0)
       (effects (font (size 1.27 1.27)) (justify left) hide)
     )
@@
     (property "Arrow Price/Stock" "" (at 231.775 153.67 0)
       (effects (font (size 1.27 1.27)) (justify left) hide)
+    )
+    (property "Extended" "0" (at 217.805 132.08 0)
+      (effects (font (size 1.27 1.27)) hide)
+    )
+    (property "Price" "0.0035" (at 217.805 132.08 0)
+      (effects (font (size 1.27 1.27)) hide)
     )
     (pin "1")
@@
       (effects (font (size 1.27 1.27)) hide)
     )
-    (property "Price" "" (at 103.505 42.545 0)
+    (property "Price" "0" (at 103.505 42.545 0)
       (effects (font (size 1.27 1.27)) hide)
     )
@@
       (effects (font (size 1.27 1.27)) hide)
     )
-    (property "Extended" "" (at 103.505 42.545 0)
+    (property "Extended" "0" (at 103.505 42.545 0)
+      (effects (font (size 1.27 1.27)) hide)
+    )
+    (property "Manufacturer_Part_Number" "0" (at 103.505 42.545 0)
       (effects (font (size 1.27 1.27)) hide)
     )
@@
       (effects (font (size 1.27 1.27)) (justify bottom) hide)
     )
-    (property "Datasheet" "" (at 27.94 92.71 0)
+    (property "Datasheet" "-" (at 27.94 92.71 0)
       (effects (font (size 1.27 1.27)) hide)
     )
@@
     )
     (property "Extended" "0" (at 27.94 92.71 0)
+      (effects (font (size 1.27 1.27)) hide)
+    )
+    (property "Description" "-" (at 27.94 92.71 0)
+      (effects (font (size 1.27 1.27)) hide)
+    )
+    (property "Manufacturer_Part_Number" "-" (at 27.94 92.71 0)
       (effects (font (size 1.27 1.27)) hide)
     )
@@
       (effects (font (size 1.27 1.27)) hide)
     )
-    (property "Price" "" (at 132.08 118.745 0)
+    (property "Price" "0" (at 132.08 118.745 0)
       (effects (font (size 1.27 1.27)) hide)
     )
@@
       (effects (font (size 1.27 1.27)) hide)
     )
-    (property "Extended" "" (at 132.08 118.745 0)
+    (property "Extended" "0" (at 132.08 118.745 0)
+      (effects (font (size 1.27 1.27)) hide)
+    )
+    (property "Manufacturer_Part_Number" "0" (at 132.08 118.745 0)
       (effects (font (size 1.27 1.27)) hide)
     )
@@
       (effects (font (size 1.27 1.27)) (justify left) hide)
     )
-    (property "Description" "Thick Film Resistors - SMD 0402 1/16W 1% 0R T/R-10000" (at 232.41 108.585 0)
+    (property "Description" "0 Resistor - 0402" (at 232.41 108.585 0)
       (effects (font (size 1.27 1.27)) (justify left) hide)
     )
@@
     (property "Arrow Price/Stock" "" (at 232.41 126.365 0)
       (effects (font (size 1.27 1.27)) (justify left) hide)
+    )
+    (property "Extended" "0" (at 218.44 104.775 0)
+      (effects (font (size 1.27 1.27)) hide)
+    )
+    (property "Price" "0.0035" (at 218.44 104.775 0)
+      (effects (font (size 1.27 1.27)) hide)
     )
     (pin "1")
@@
       (effects (font (size 1.27 1.27)) hide)
     )
-    (property "Price" "" (at 206.375 132.08 0)
+    (property "Price" "0" (at 206.375 132.08 0)
       (effects (font (size 1.27 1.27)) hide)
     )
@@
       (effects (font (size 1.27 1.27)) hide)
     )
-    (property "Extended" "" (at 206.375 132.08 0)
+    (property "Extended" "0" (at 206.375 132.08 0)
+      (effects (font (size 1.27 1.27)) hide)
+    )
+    (property "Manufacturer_Part_Number" "0" (at 206.375 132.08 0)
       (effects (font (size 1.27 1.27)) hide)
     )
@@
       (effects (font (size 1.27 1.27)) (justify left) hide)
     )
-    (property "Description" "Thick Film Resistors - SMD 0402 1/16W 1% 0R T/R-10000" (at 151.13 122.555 0)
+    (property "Description" "0 Resistor - 0402" (at 151.13 122.555 0)
       (effects (font (size 1.27 1.27)) (justify left) hide)
     )
@@
     (property "Arrow Price/Stock" "" (at 151.13 140.335 0)
       (effects (font (size 1.27 1.27)) (justify left) hide)
+    )
+    (property "Extended" "0" (at 137.16 118.745 0)
+      (effects (font (size 1.27 1.27)) hide)
+    )
+    (property "Price" "0.0035" (at 137.16 118.745 0)
+      (effects (font (size 1.27 1.27)) hide)
     )
     (pin "1")
@@
       (effects (font (size 1.27 1.27)) (justify left) hide)
     )
-    (property "Description" "Thick Film Resistors - SMD 0402 1/16W 1% 0R T/R-10000" (at 129.54 46.355 0)
+    (property "Description" "0 Resistor - 0402" (at 129.54 46.355 0)
       (effects (font (size 1.27 1.27)) (justify left) hide)
     )
@@
     (property "Arrow Price/Stock" "" (at 129.54 64.135 0)
       (effects (font (size 1.27 1.27)) (justify left) hide)
+    )
+    (property "Extended" "0" (at 115.57 42.545 0)
+      (effects (font (size 1.27 1.27)) hide)
+    )
+    (property "Price" "0.0035" (at 115.57 42.545 0)
+      (effects (font (size 1.27 1.27)) hide)
     )
     (pin "1")
@@
       (effects (font (size 1.27 1.27)) hide)
     )
-    (property "Price" "" (at 205.74 104.775 0)
+    (property "Price" "0" (at 205.74 104.775 0)
       (effects (font (size 1.27 1.27)) hide)
     )
@@
       (effects (font (size 1.27 1.27)) hide)
     )
-    (property "Extended" "" (at 205.74 104.775 0)
+    (property "Extended" "0" (at 205.74 104.775 0)
+      (effects (font (size 1.27 1.27)) hide)
+    )
+    (property "Manufacturer_Part_Number" "0" (at 205.74 104.775 0)
       (effects (font (size 1.27 1.27)) hide)
     )
@@
       (effects (font (size 1.27 1.27)) (justify left) hide)
     )
-    (property "Description" "Thick Film Resistors - SMD 0402 1/16W 1% 0R T/R-10000" (at 69.215 113.03 0)
+    (property "Description" "0 Resistor - 0402" (at 69.215 113.03 0)
       (effects (font (size 1.27 1.27)) (justify left) hide)
     )
@@
     (property "Arrow Price/Stock" "" (at 69.215 130.81 0)
       (effects (font (size 1.27 1.27)) (justify left) hide)
+    )
+    (property "Extended" "0" (at 55.245 109.22 0)
+      (effects (font (size 1.27 1.27)) hide)
+    )
+    (property "Price" "0.0035" (at 55.245 109.22 0)
+      (effects (font (size 1.27 1.27)) hide)
     )
     (pin "1")
@@
       (effects (font (size 1.27 1.27)) hide)
     )
-    (property "Price" "" (at 44.45 109.22 0)
+    (property "Price" "0" (at 44.45 109.22 0)
       (effects (font (size 1.27 1.27)) hide)
     )
@@
       (effects (font (size 1.27 1.27)) hide)
     )
-    (property "Extended" "" (at 44.45 109.22 0)
+    (property "Extended" "0" (at 44.45 109.22 0)
+      (effects (font (size 1.27 1.27)) hide)
+    )
+    (property "Manufacturer_Part_Number" "0" (at 44.45 109.22 0)
       (effects (font (size 1.27 1.27)) hide)
     )
@@
       (effects (font (size 1.27 1.27)) (justify bottom) hide)
     )
-    (property "Datasheet" "" (at 48.26 118.11 0)
+    (property "Datasheet" "-" (at 48.26 118.11 0)
       (effects (font (size 1.27 1.27)) hide)
     )
@@
       (effects (font (size 1.27 1.27)) (justify bottom) hide)
     )
-    (property "Price" "" (at 48.26 118.11 0)
+    (property "Price" "-" (at 48.26 118.11 0)
       (effects (font (size 1.27 1.27)) hide)
     )
@@
       (effects (font (size 1.27 1.27)) hide)
     )
-    (property "Extended" "" (at 48.26 118.11 0)
-      (effects (font (size 1.27 1.27)) hide)
-    )
+    (property "Extended" "-" (at 48.26 118.11 0)
+      (effects (font (size 1.27 1.27)) hide)
+    )
+    (property "Description" "-" (at 48.26 118.11 0)
+      (effects (font (size 1.27 1.27)) hide)
+    )
+    (property "Manufacturer_Part_Number" "-" (at 48.26 118.11 0)
+      (effects (font (size 1.27 1.27)) hide)
+    )

Commit message: BOM Update
Parts:
- D1: Extended - -> 0
Changed lines of the file:
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@@
+      (effects (font (size 1.27 1.27)) hide)
+    )
+    (property "Description" "Voltage Regulator IC" (at 186.055 107.315 0)
       (effects (font (size 1.27 1.27)) hide)
     )
@@
       (effects (font (size 1.27 1.27)) hide)
     )
+    (property "Description" "Voltage Regulator IC" (at 186.055 134.62 0)
+      (effects (font (size 1.27 1.27)) hide)
+    )
     (pin "1")
     (pin "2")
@@
       (effects (font (size 1.27 1.27)) (justify left) hide)
     )
-    (property "Description" "1K Resistor - 0402" (at 96.52 40.005 0)
+    (property "Description" "1k Resistor - 0805" (at 96.52 40.005 0)
       (effects (font (size 1.27 1.27)) (justify left) hide)
     )
@@
       (effects (font (size 1.27 1.27)) hide)
     )
+    (property "Description" "Test Point (DNP)" (at 103.505 42.545 0)
+      (effects (font (size 1.27 1.27)) hide)
+    )
     (pin "1")
     (instances
@@
       (effects (font (size 1.27 1.27)) hide)
     )
-    (property "Description" "-" (at 27.94 92.71 0)
+    (property "Description" "Battery Holder" (at 27.94 92.71 0)
       (effects (font (size 1.27 1.27)) hide)
     )
@@
       (effects (font (size 1.27 1.27)) hide)
     )
+    (property "Description" "Test Point (DNP)" (at 132.08 118.745 0)
+      (effects (font (size 1.27 1.27)) hide)
+    )
     (pin "1")
     (instances
@@
     )
     (property "Manufacturer_Part_Number" "0" (at 206.375 132.08 0)
+      (effects (font (size 1.27 1.27)) hide)
+    )
+    (property "Description" "Test Point (DNP)" (at 206.375 132.08 0)
       (effects (font (size 1.27 1.27)) hide)
     )
@@
     )
     (property "Manufacturer_Part_Number" "0" (at 205.74 104.775 0)
+      (effects (font (size 1.27 1.27)) hide)
+    )
+    (property "Description" "Test Point (DNP)" (at 205.74 104.775 0)
       (effects (font (size 1.27 1.27)) hide)
     )
@@
       (effects (font (size 1.27 1.27)) (justify left) hide)
     )
-    (property "Description" "1k Resistor - 0402" (at 19.05 60.96 0)
+    (property "Description" "1k Resistor - 0805" (at 19.05 60.96 0)
       (effects (font (size 1.27 1.27)) (justify left) hide)
     )
@@
       (effects (font (size 1.27 1.27)) hide)
     )
+    (property "Description" "Test Point (DNP)" (at 44.45 109.22 0)
+      (effects (font (size 1.27 1.27)) hide)
+    )
     (pin "1")
     (instances
@@
       (effects (font (size 1.27 1.27)) hide)
     )
-    (property "Extended" "-" (at 48.26 118.11 0)
-      (effects (font (size 1.27 1.27)) hide)
-    )
-    (property "Description" "-" (at 48.26 118.11 0)
-      (effects (font (size 1.27 1.27)) hide)
-    )
+    (property "Extended" "0" (at 48.26 118.11 0)
+      (effects (font (size 1.27 1.27)) hide)
+    )
+    (property "Description" "Zener Diode" (at 48.26 118.11 0)
+      (effects (font (size 1.27 1.27)) hide)
+    )
