File: EEE3088/Power_kicad_sch.kicad_sch (KiCad schematic)
At the start: 28 parts, among them U1 TP4056, U2 HT7533-1

Commit message: Light update to power
Other:
- moved on the sheet: N-Mos1, R10, R7, R8, R9, TP3, TP4, TP5, U2, Voltage-Regulator-1

Commit message: power
Connections:
- net 5V renamed +5V
Changed lines of the file:
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@@
   (junction (at 90.805 116.84) (diameter 0) (color 0 0 0 0)
   )
-  (junction (at 48.895 24.765) (diameter 0) (color 0 0 0 0)
-  )
   (junction (at 81.915 24.765) (diameter 0) (color 0 0 0 0)
   )
@@
   )
   (junction (at 213.995 132.08) (diameter 0) (color 0 0 0 0)
+  )
+  (junction (at 55.88 24.765) (diameter 0) (color 0 0 0 0)
   )
   (junction (at 44.45 109.22) (diameter 0) (color 0 0 0 0)
@@
     (stroke (width 0) (type default))
   )
-  (wire (pts (xy 48.895 22.225) (xy 48.895 24.765))
-    (stroke (width 0) (type default))
-  )
   (wire (pts (xy 27.94 100.33) (xy 27.94 109.22))
     (stroke (width 0) (type default))
@@
     (stroke (width 0) (type default))
   )
-  (wire (pts (xy 40.64 24.765) (xy 48.895 24.765))
-    (stroke (width 0) (type default))
-  )
   (wire (pts (xy 247.015 104.775) (xy 243.84 104.775))
     (stroke (width 0) (type default))
@@
     (stroke (width 0) (type default))
   )
-  (wire (pts (xy 48.895 24.765) (xy 81.915 24.765))
+  (wire (pts (xy 40.64 24.765) (xy 55.88 24.765))
     (stroke (width 0) (type default))
   )
@@
   )
   (wire (pts (xy 40.64 45.085) (xy 40.64 40.64))
+    (stroke (width 0) (type default))
+  )
+  (wire (pts (xy 55.88 24.765) (xy 81.915 24.765))
     (stroke (width 0) (type default))
   )
@@
     )
   )
-  (global_label "5V" (shape input) (at 48.895 22.225 0) (fields_autoplaced)
-    (effects (font (size 1.27 1.27)) (justify left))
-    (property "Intersheetrefs" "${INTERSHEET_REFS}" (at 54.0989 22.225 0)
-      (effects (font (size 1.27 1.27)) (justify left) hide)
-    )
-  )
   (symbol (lib_id "power:GND") (at 193.675 112.395 0) (unit 1)
     (in_bom yes) (on_board yes) (dnp no) (fields_autoplaced)
@@
         )
       )
+    )
+  )
+  (symbol (lib_id "power:+5V") (at 55.88 24.765 0) (unit 1)
+    (in_bom yes) (on_board yes) (dnp no) (fields_autoplaced)
+    (property "Reference" "#PWR045" (at 55.88 28.575 0)
+      (effects (font (size 1.27 1.27)) hide)
+    )
+    (property "Value" "+5V" (at 55.88 21.59 0)
+      (effects (font (size 1.27 1.27)))
+    )
+    (property "Footprint" "" (at 55.88 24.765 0)
+      (effects (font (size 1.27 1.27)) hide)
+    )
+    (property "Datasheet" "" (at 55.88 24.765 0)
+      (effects (font (size 1.27 1.27)) hide)
+    )
+    (pin "1")
+    (instances
+      (project "EEE3088"
+        (path "/83bdd5e1-981a-4ca1-9a2f-70dea9f00850/1213f935-6f8d-4a20-9c2e-6b5e9a834fe6"
+          (reference "#PWR045") (unit 1)
+        )
+      )

Commit message: attempt to assign footprints
Parts:
- BT1: footprint BAT_BH-18650-PC -> (none)
- C1, C2: footprint CAPC1608X90N -> (none)
- LED1: footprint LEDC1608X70N -> (none)
- LED2: footprint LEDC1608X50N -> (none)
- N-Mos1, P-Mos1: footprint SOT95P280X125-3N -> (none)
- Op-Amp1: footprint SOIC127P600X175-8N -> (none)
- R1, R10, R4, R6, R8, R9: footprint RESC1005X40N -> (none)
- R2: footprint RESC1608X55N -> (none)
- R5: footprint RESC3116X65N -> (none)
- R7: footprint RESC2013X65N -> (none)
- U1: footprint SOP127P600X175-9N -> (none)
- U2, Voltage-Regulator-1: footprint SOT89 -> (none)
- Z1: footprint SODFL2513X100N -> MyZener:SODFL2513X100N
Changed lines of the file:
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@@
       (effects (font (size 1.27 1.27)) (justify left))
     )
-    (property "Footprint" "RESC2013X65N" (at 144.78 135.255 0)
+    (property "Footprint" "" (at 144.78 135.255 0)
       (effects (font (size 1.27 1.27)) (justify left) hide)
     )
@@
       (effects (font (size 1.27 1.27)))
     )
-    (property "Footprint" "SOT89" (at 193.675 107.315 0)
+    (property "Footprint" "" (at 193.675 107.315 0)
       (effects (font (size 1.27 1.27)) (justify bottom) hide)
     )
@@
       (effects (font (size 1.27 1.27)))
     )
-    (property "Footprint" "SOT89" (at 193.675 134.62 0)
+    (property "Footprint" "" (at 193.675 134.62 0)
       (effects (font (size 1.27 1.27)) (justify bottom) hide)
     )
@@
       (effects (font (size 1.27 1.27)) (justify right))
     )
-    (property "Footprint" "RESC3116X65N" (at 36.83 129.54 0)
+    (property "Footprint" "" (at 36.83 129.54 0)
       (effects (font (size 1.27 1.27)) (justify left) hide)
     )
@@
       (effects (font (size 1.27 1.27)) (justify left))
     )
-    (property "Footprint" "RESC1005X40N" (at 101.6 40.005 0)
+    (property "Footprint" "" (at 101.6 40.005 0)
       (effects (font (size 1.27 1.27)) (justify left) hide)
     )
@@
       (effects (font (size 1.27 1.27)) (justify left))
     )
-    (property "Footprint" "SOT95P280X125-3N" (at 147.32 110.49 0)
+    (property "Footprint" "" (at 147.32 110.49 0)
       (effects (font (size 1.27 1.27)) (justify left) hide)
     )
@@
       (effects (font (size 1.27 1.27)))
     )
-    (property "Footprint" "RESC1005X40N" (at 239.395 130.81 0)
+    (property "Footprint" "" (at 239.395 130.81 0)
       (effects (font (size 1.27 1.27)) (justify left) hide)
     )
@@
       (effects (font (size 1.27 1.27)))
     )
-    (property "Footprint" "CAPC1608X90N" (at 22.86 31.115 0)
+    (property "Footprint" "" (at 22.86 31.115 0)
       (effects (font (size 1.27 1.27)) (justify bottom) hide)
     )
@@
       (effects (font (size 1.27 1.27)) (justify left))
     )
-    (property "Footprint" "SODFL2513X100N" (at -45.39 120.65 0)
+    (property "Footprint" "MyZener:SODFL2513X100N" (at -45.39 120.65 0)
       (effects (font (size 1.27 1.27)) (justify left top) hide)
     )
@@
       (effects (font (size 1.27 1.27)))
     )
-    (property "Footprint" "LEDC1608X70N" (at 38.1 36.83 0)
+    (property "Footprint" "" (at 38.1 36.83 0)
       (effects (font (size 1.27 1.27)) (justify left bottom) hide)
     )
@@
       (effects (font (size 1.27 1.27)) (justify right))
     )
-    (property "Footprint" "BAT_BH-18650-PC" (at 27.94 92.71 0)
+    (property "Footprint" "" (at 27.94 92.71 0)
       (effects (font (size 1.27 1.27)) (justify bottom) hide)
     )
@@
       (effects (font (size 1.27 1.27)))
     )
-    (property "Footprint" "RESC1005X40N" (at 240.03 103.505 0)
+    (property "Footprint" "" (at 240.03 103.505 0)
       (effects (font (size 1.27 1.27)) (justify left) hide)
     )
@@
       (effects (font (size 1.27 1.27)))
     )
-    (property "Footprint" "RESC1005X40N" (at 160.655 117.475 0)
+    (property "Footprint" "" (at 160.655 117.475 0)
       (effects (font (size 1.27 1.27)) (justify left) hide)
     )
@@
       (effects (font (size 1.27 1.27)) (justify right))
     )
-    (property "Footprint" "CAPC1608X90N" (at 88.265 53.34 0)
+    (property "Footprint" "" (at 88.265 53.34 0)
       (effects (font (size 1.27 1.27)) (justify bottom) hide)
     )
@@
       (effects (font (size 1.27 1.27)))
     )
-    (property "Footprint" "RESC1005X40N" (at 129.54 41.275 0)
+    (property "Footprint" "" (at 129.54 41.275 0)
       (effects (font (size 1.27 1.27)) (justify left) hide)
     )
@@
       (effects (font (size 1.27 1.27)))
     )
-    (property "Footprint" "RESC1005X40N" (at 69.215 107.95 0)
+    (property "Footprint" "" (at 69.215 107.95 0)
       (effects (font (size 1.27 1.27)) (justify left) hide)
     )
@@
       (effects (font (size 1.27 1.27)))
     )
-    (property "Footprint" "SOP127P600X175-9N" (at 66.675 47.625 0)
+    (property "Footprint" "" (at 66.675 47.625 0)
       (effects (font (size 1.27 1.27)) (justify bottom) hide)
     )
@@
       (effects (font (size 1.27 1.27)))
     )
-    (property "Footprint" "LEDC1608X50N" (at 87.63 28.575 0)
+    (property "Footprint" "" (at 87.63 28.575 0)
       (effects (font (size 1.27 1.27)) (justify left bottom) hide)
     )
@@
       (effects (font (size 1.27 1.27)) (justify left))
     )
-    (property "Footprint" "RESC1005X40N" (at 24.13 60.96 0)
+    (property "Footprint" "" (at 24.13 60.96 0)
       (effects (font (size 1.27 1.27)) (justify left) hide)
     )
@@
       (effects (font (size 1.27 1.27)))
     )
-    (property "Footprint" "SOT95P280X125-3N" (at 39.37 105.41 0)
+    (property "Footprint" "" (at 39.37 105.41 0)
       (effects (font (size 1.27 1.27)) (justify left) hide)
     )
@@
       (effects (font (size 1.27 1.27)) (justify left))
     )
-    (property "Footprint" "SOIC127P600X175-8N" (at 120.65 99.06 0)
+    (property "Footprint" "" (at 120.65 99.06 0)
       (effects (font (size 1.27 1.27)) (justify left) hide)
     )
@@
       (effects (font (size 1.27 1.27)))
     )
-    (property "Footprint" "RESC1608X55N" (at 43.815 48.895 0)
-      (effects (font (size 1.27 1.27)) (justify left) hide)
-    )
+    (property "Footprint" "" (at 43.815 48.895 0)
+      (effects (font (size 1.27 1.27)) (justify left) hide)
+    )

Commit message: adding footprints power
Parts:
- BT1: footprint (none) -> BH-18650-PC:BAT_BH-18650-PC
- C1, C2: footprint (none) -> CL10A106KP8NNNC:CAPC1608X90N
- LED1: footprint (none) -> MyRedLED:LEDC1608X70N
- LED2: footprint (none) -> MyGreenLED:LEDC1608X50N
- N-Mos1: footprint (none) -> MyNmos:SOT95P280X125-3N
- Op-Amp1: footprint (none) -> Myopamp:SOIC127P600X175-8N
- P-Mos1: footprint (none) -> MyPmos:SOT95P280X125-3N
- R10, R4, R6, R8, R9: footprint (none) -> My0R:RESC1005X40N
- R2: footprint (none) -> My1.2k:RESC1608X55N
- R5: footprint (none) -> My100k:RESC3116X65N
- R7: footprint (none) -> My1M:RESC2013X65N
- U1: footprint (none) -> TP4056:SOP127P600X175-9N
- U2, Voltage-Regulator-1: footprint (none) -> HT7533-1:SOT89
Changed lines of the file:
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@@
       (effects (font (size 1.27 1.27)) (justify left))
     )
-    (property "Footprint" "" (at 144.78 135.255 0)
+    (property "Footprint" "My1M:RESC2013X65N" (at 144.78 135.255 0)
       (effects (font (size 1.27 1.27)) (justify left) hide)
     )
@@
       (effects (font (size 1.27 1.27)))
     )
-    (property "Footprint" "" (at 193.675 107.315 0)
+    (property "Footprint" "HT7533-1:SOT89" (at 193.675 107.315 0)
       (effects (font (size 1.27 1.27)) (justify bottom) hide)
     )
@@
       (effects (font (size 1.27 1.27)))
     )
-    (property "Footprint" "" (at 193.675 134.62 0)
+    (property "Footprint" "HT7533-1:SOT89" (at 193.675 134.62 0)
       (effects (font (size 1.27 1.27)) (justify bottom) hide)
     )
@@
       (effects (font (size 1.27 1.27)) (justify right))
     )
-    (property "Footprint" "" (at 36.83 129.54 0)
+    (property "Footprint" "My100k:RESC3116X65N" (at 36.83 129.54 0)
       (effects (font (size 1.27 1.27)) (justify left) hide)
     )
@@
       (effects (font (size 1.27 1.27)) (justify left))
     )
-    (property "Footprint" "" (at 147.32 110.49 0)
+    (property "Footprint" "MyNmos:SOT95P280X125-3N" (at 147.32 110.49 0)
       (effects (font (size 1.27 1.27)) (justify left) hide)
     )
@@
       (effects (font (size 1.27 1.27)))
     )
-    (property "Footprint" "" (at 239.395 130.81 0)
+    (property "Footprint" "My0R:RESC1005X40N" (at 239.395 130.81 0)
       (effects (font (size 1.27 1.27)) (justify left) hide)
     )
@@
       (effects (font (size 1.27 1.27)))
     )
-    (property "Footprint" "" (at 22.86 31.115 0)
+    (property "Footprint" "CL10A106KP8NNNC:CAPC1608X90N" (at 22.86 31.115 0)
       (effects (font (size 1.27 1.27)) (justify bottom) hide)
     )
@@
       (effects (font (size 1.27 1.27)))
     )
-    (property "Footprint" "" (at 38.1 36.83 0)
+    (property "Footprint" "MyRedLED:LEDC1608X70N" (at 38.1 36.83 0)
       (effects (font (size 1.27 1.27)) (justify left bottom) hide)
     )
@@
       (effects (font (size 1.27 1.27)) (justify right))
     )
-    (property "Footprint" "" (at 27.94 92.71 0)
+    (property "Footprint" "BH-18650-PC:BAT_BH-18650-PC" (at 27.94 92.71 0)
       (effects (font (size 1.27 1.27)) (justify bottom) hide)
     )
@@
       (effects (font (size 1.27 1.27)))
     )
-    (property "Footprint" "" (at 240.03 103.505 0)
+    (property "Footprint" "My0R:RESC1005X40N" (at 240.03 103.505 0)
       (effects (font (size 1.27 1.27)) (justify left) hide)
     )
@@
       (effects (font (size 1.27 1.27)))
     )
-    (property "Footprint" "" (at 160.655 117.475 0)
+    (property "Footprint" "My0R:RESC1005X40N" (at 160.655 117.475 0)
       (effects (font (size 1.27 1.27)) (justify left) hide)
     )
@@
       (effects (font (size 1.27 1.27)) (justify right))
     )
-    (property "Footprint" "" (at 88.265 53.34 0)
+    (property "Footprint" "CL10A106KP8NNNC:CAPC1608X90N" (at 88.265 53.34 0)
       (effects (font (size 1.27 1.27)) (justify bottom) hide)
     )
@@
       (effects (font (size 1.27 1.27)))
     )
-    (property "Footprint" "" (at 129.54 41.275 0)
+    (property "Footprint" "My0R:RESC1005X40N" (at 129.54 41.275 0)
       (effects (font (size 1.27 1.27)) (justify left) hide)
     )
@@
       (effects (font (size 1.27 1.27)))
     )
-    (property "Footprint" "" (at 69.215 107.95 0)
+    (property "Footprint" "My0R:RESC1005X40N" (at 69.215 107.95 0)
       (effects (font (size 1.27 1.27)) (justify left) hide)
     )
@@
       (effects (font (size 1.27 1.27)))
     )
-    (property "Footprint" "" (at 66.675 47.625 0)
+    (property "Footprint" "TP4056:SOP127P600X175-9N" (at 66.675 47.625 0)
       (effects (font (size 1.27 1.27)) (justify bottom) hide)
     )
@@
       (effects (font (size 1.27 1.27)))
     )
-    (property "Footprint" "" (at 87.63 28.575 0)
+    (property "Footprint" "MyGreenLED:LEDC1608X50N" (at 87.63 28.575 0)
       (effects (font (size 1.27 1.27)) (justify left bottom) hide)
     )
@@
       (effects (font (size 1.27 1.27)))
     )
-    (property "Footprint" "" (at 39.37 105.41 0)
+    (property "Footprint" "MyPmos:SOT95P280X125-3N" (at 39.37 105.41 0)
       (effects (font (size 1.27 1.27)) (justify left) hide)
     )
@@
       (effects (font (size 1.27 1.27)) (justify left))
     )
-    (property "Footprint" "" (at 120.65 99.06 0)
+    (property "Footprint" "Myopamp:SOIC127P600X175-8N" (at 120.65 99.06 0)
       (effects (font (size 1.27 1.27)) (justify left) hide)
     )
@@
   )
   (symbol (lib_id "0603WAF1201T5E:0603WAF1201T5E") (at 29.845 50.165 0) (unit 1)
-    (in_bom yes) (on_board yes) (dnp no) (fields_autoplaced)
+    (in_bom yes) (on_board yes) (dnp no)
     (property "Reference" "R2" (at 38.735 45.085 0)
       (effects (font (size 1.27 1.27)))
@@
       (effects (font (size 1.27 1.27)))
     )
-    (property "Footprint" "" (at 43.815 48.895 0)
-      (effects (font (size 1.27 1.27)) (justify left) hide)
-    )
+    (property "Footprint" "My1.2k:RESC1608X55N" (at 32.385 58.42 0)
+      (effects (font (size 1.27 1.27)) (justify left) hide)
+    )

Commit message: power
Parts:
- removed R1: 1k, symbol 0402WGF1001TCE:0402WGF1001TCE
- added R32: 1k, RESC1608X55N, symbol my 1k:0603WAF1001T5E
- TP1, TP2, TP22, TP3, TP4, TP5: footprint (none) -> TestPoint:TestPoint_Keystone_5005-5009_Compact
Connections:
- net at LED1.1: now also R32.2
- net at U1.7 (~{CHRG}): now also R32.1
Changed lines of the file:
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@@
       (effects (font (size 1.27 1.27)) (justify left))
     )
-    (property "Footprint" "" (at 108.585 42.545 0)
+    (property "Footprint" "TestPoint:TestPoint_Keystone_5005-5009_Compact" (at 108.585 42.545 0)
       (effects (font (size 1.27 1.27)) hide)
     )
@@
       (effects (font (size 1.27 1.27)) (justify left))
     )
-    (property "Footprint" "" (at 129.54 109.22 0)
+    (property "Footprint" "TestPoint:TestPoint_Keystone_5005-5009_Compact" (at 129.54 109.22 0)
       (effects (font (size 1.27 1.27)) hide)
     )
@@
       (effects (font (size 1.27 1.27)))
     )
-    (property "Footprint" "" (at 141.605 113.665 0)
+    (property "Footprint" "TestPoint:TestPoint_Keystone_5005-5009_Compact" (at 141.605 113.665 0)
       (effects (font (size 1.27 1.27)) hide)
     )
@@
       (effects (font (size 1.27 1.27)) (justify left))
     )
-    (property "Footprint" "" (at 219.075 132.08 0)
+    (property "Footprint" "TestPoint:TestPoint_Keystone_5005-5009_Compact" (at 219.075 132.08 0)
       (effects (font (size 1.27 1.27)) hide)
     )
@@
       (effects (font (size 1.27 1.27)) (justify left))
     )
-    (property "Footprint" "" (at 218.44 104.775 0)
+    (property "Footprint" "TestPoint:TestPoint_Keystone_5005-5009_Compact" (at 218.44 104.775 0)
       (effects (font (size 1.27 1.27)) hide)
     )
@@
     )
   )
-  (symbol (lib_id "0402WGF1001TCE:0402WGF1001TCE") (at 22.86 46.99 270) (unit 1)
-    (in_bom yes) (on_board yes) (dnp no) (fields_autoplaced)
-    (property "Reference" "R1" (at 26.035 55.245 90)
-      (effects (font (size 1.27 1.27)) (justify left))
-    )
-    (property "Value" "1k" (at 26.035 57.785 90)
-      (effects (font (size 1.27 1.27)) (justify left))
-    )
-    (property "Footprint" "" (at 24.13 60.96 0)
-      (effects (font (size 1.27 1.27)) (justify left) hide)
-    )
-    (property "Datasheet" "https://datasheet.lcsc.com/szlcsc/Uniroyal-Elec-0402WGF1001TCE_C11702.pdf" (at 21.59 60.96 0)
-      (effects (font (size 1.27 1.27)) (justify left) hide)
-    )
-    (property "Description" "1k Resistor - 0805" (at 19.05 60.96 0)
-      (effects (font (size 1.27 1.27)) (justify left) hide)
-    )
-    (property "Height" "0.4" (at 16.51 60.96 0)
-      (effects (font (size 1.27 1.27)) (justify left) hide)
-    )
-    (property "Manufacturer_Name" "UNI-ROYAL(Uniroyal Elec)" (at 13.97 60.96 0)
-      (effects (font (size 1.27 1.27)) (justify left) hide)
-    )
-    (property "Manufacturer_Part_Number" "0805W8F1801T5E" (at 11.43 60.96 0)
-      (effects (font (size 1.27 1.27)) (justify left) hide)
-    )
-    (property "Mouser Part Number" "" (at 8.89 60.96 0)
-      (effects (font (size 1.27 1.27)) (justify left) hide)
-    )
-    (property "Mouser Price/Stock" "" (at 6.35 60.96 0)
-      (effects (font (size 1.27 1.27)) (justify left) hide)
-    )
-    (property "Arrow Part Number" "" (at 3.81 60.96 0)
-      (effects (font (size 1.27 1.27)) (justify left) hide)
-    )
-    (property "Arrow Price/Stock" "" (at 1.27 60.96 0)
-      (effects (font (size 1.27 1.27)) (justify left) hide)
-    )
-    (property "Price" "0.0018" (at 22.86 46.99 0)
-      (effects (font (size 1.27 1.27)) hide)
-    )
-    (property "Basic" "" (at 22.86 46.99 0)
-      (effects (font (size 1.27 1.27)) hide)
-    )
-    (property "Extended" "0" (at 22.86 46.99 0)
-      (effects (font (size 1.27 1.27)) hide)
-    )
-    (property "JLC Part Number" "C17398" (at 22.86 46.99 0)
-      (effects (font (size 1.27 1.27)) hide)
-    )
-    (pin "1")
-    (pin "2")
-    (instances
-      (project "Power_kicad_sch"
-        (path "/02e53f89-135a-4459-982b-e3c28e008824"
-          (reference "R1") (unit 1)
-        )
-      )
-      (project "EEE3088"
-        (path "/83bdd5e1-981a-4ca1-9a2f-70dea9f00850/1213f935-6f8d-4a20-9c2e-6b5e9a834fe6"
-          (reference "R1") (unit 1)
-        )
-      )
-    )
-  )
   (symbol (lib_id "Connector:TestPoint") (at 44.45 109.22 0) (unit 1)
     (in_bom yes) (on_board yes) (dnp no) (fields_autoplaced)
@@
       (effects (font (size 1.27 1.27)) (justify left))
     )
-    (property "Footprint" "" (at 49.53 109.22 0)
+    (property "Footprint" "TestPoint:TestPoint_Keystone_5005-5009_Compact" (at 49.53 109.22 0)
       (effects (font (size 1.27 1.27)) hide)
     )
@@
         )
       )
+    )
+  )
+  (symbol (lib_id "my 1k:0603WAF1001T5E") (at 22.86 64.77 90) (unit 1)
+    (in_bom yes) (on_board yes) (dnp no) (fields_autoplaced)
+    (property "Reference" "R32" (at 25.4 55.245 90)
+      (effects (font (size 1.27 1.27)) (justify right))
+    )
+    (property "Value" "1k" (at 25.4 57.785 90)
+      (effects (font (size 1.27 1.27)) (justify right))
+    )
+    (property "Footprint" "RESC1608X55N" (at 21.59 50.8 0)
+      (effects (font (size 1.27 1.27)) (justify left) hide)
+    )
+    (property "Datasheet" "https://datasheet.lcsc.com/szlcsc/Uniroyal-Elec-0603WAF1001T5E_C21190.pdf" (at 24.13 50.8 0)
+      (effects (font (size 1.27 1.27)) (justify left) hide)
+    )
+    (property "Description" "1k Resistor" (at 26.67 50.8 0)
+      (effects (font (size 1.27 1.27)) (justify left) hide)
+    )
+    (property "Height" "0.55" (at 29.21 50.8 0)
+      (effects (font (size 1.27 1.27)) (justify left) hide)
+    )
+    (property "Manufacturer_Name" "UNI-ROYAL(Uniroyal Elec)" (at 31.75 50.8 0)
+      (effects (font (size 1.27 1.27)) (justify left) hide)
+    )
+    (property "Manufacturer_Part_Number" "0603WAF1001T5E" (at 34.29 50.8 0)
+      (effects (font (size 1.27 1.27)) (justify left) hide)
+    )
+    (property "Mouser Part Number" "" (at 36.83 50.8 0)
+      (effects (font (size 1.27 1.27)) (justify left) hide)
+    )
+    (property "Mouser Price/Stock" "" (at 39.37 50.8 0)
+      (effects (font (size 1.27 1.27)) (justify left) hide)
+    )
+    (property "Arrow Part Number" "" (at 41.91 50.8 0)
+      (effects (font (size 1.27 1.27)) (justify left) hide)
+    )
+    (property "Arrow Price/Stock" "" (at 44.45 50.8 0)
+      (effects (font (size 1.27 1.27)) (justify left) hide)
+    )
+    (property "Extended" "0" (at 22.86 64.77 0)
+      (effects (font (size 1.27 1.27)) hide)
+    )
+    (property "JLC Part Number" "C21190" (at 22.86 64.77 0)
+      (effects (font (size 1.27 1.27)) hide)
+    )
+    (property "Price" "0.0006" (at 22.86 64.77 0)
+      (effects (font (size 1.27 1.27)) hide)
+    )
+    (pin "1")
+    (pin "2")
+    (instances
+      (project "EEE3088"
+        (path "/83bdd5e1-981a-4ca1-9a2f-70dea9f00850/1213f935-6f8d-4a20-9c2e-6b5e9a834fe6"
+          (reference "R32") (unit 1)
+        )
+      )

Commit message: power
Parts:
- R4: footprint (none) -> RESC1608X55N; JLC Part Number C17398 -> C21190; Manufacturer_Part_Number 0805W8F1801T5E -> 0603WAF1001T5E; Price 0.0018 -> 0.0006
Changed lines of the file:
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@@
       (effects (font (size 1.27 1.27)) (justify left))
     )
-    (property "Footprint" "" (at 101.6 40.005 0)
+    (property "Footprint" "RESC1608X55N" (at 101.6 40.005 0)
       (effects (font (size 1.27 1.27)) (justify left) hide)
     )
-    (property "Datasheet" "https://datasheet.lcsc.com/szlcsc/Uniroyal-Elec-0402WGF1001TCE_C11702.pdf" (at 99.06 40.005 0)
+    (property "Datasheet" "https://datasheet.lcsc.com/szlcsc/Uniroyal-Elec-0603WAF1001T5E_C21190.pdf" (at 99.06 40.005 0)
       (effects (font (size 1.27 1.27)) (justify left) hide)
     )
@@
       (effects (font (size 1.27 1.27)) (justify left) hide)
     )
-    (property "Manufacturer_Part_Number" "0805W8F1801T5E" (at 88.9 40.005 0)
+    (property "Manufacturer_Part_Number" "0603WAF1001T5E" (at 88.9 40.005 0)
       (effects (font (size 1.27 1.27)) (justify left) hide)
     )
@@
       (effects (font (size 1.27 1.27)) (justify left) hide)
     )
-    (property "Price" "0.0018" (at 100.33 26.035 0)
+    (property "Price" "0.0006" (at 100.33 26.035 0)
       (effects (font (size 1.27 1.27)) hide)
     )
@@
       (effects (font (size 1.27 1.27)) hide)
     )
-    (property "JLC Part Number" "C17398" (at 100.33 26.035 0)
+    (property "JLC Part Number" "C21190" (at 100.33 26.035 0)
       (effects (font (size 1.27 1.27)) hide)
     )
