File: EEE3088/Power_kicad_sch.kicad_sch (KiCad schematic)
At the start: 28 parts, among them U1 TP4056, U2 HT7533-1

Commit message: pcb_Sense_Initial
Parts:
- R10, R4, R6, R8, R9: footprint My0R:RESC1005X40N -> Resistor_SMD:R_0402_1005Metric
- TP1, TP2, TP22, TP3, TP4, TP5: footprint TestPoint:TestPoint_Keystone_5005-5009_Compact -> TestPoint:TestPoint_Pad_2.0x2.0mm
Changed lines of the file:
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@@
       (effects (font (size 1.27 1.27)))
     )
-    (property "Footprint" "My0R:RESC1005X40N" (at 239.395 130.81 0)
+    (property "Footprint" "Resistor_SMD:R_0402_1005Metric" (at 239.395 130.81 0)
       (effects (font (size 1.27 1.27)) (justify left) hide)
     )
@@
       (effects (font (size 1.27 1.27)) (justify left))
     )
-    (property "Footprint" "TestPoint:TestPoint_Keystone_5005-5009_Compact" (at 108.585 42.545 0)
+    (property "Footprint" "TestPoint:TestPoint_Pad_2.0x2.0mm" (at 108.585 42.545 0)
       (effects (font (size 1.27 1.27)) hide)
     )
@@
       (effects (font (size 1.27 1.27)) (justify left))
     )
-    (property "Footprint" "TestPoint:TestPoint_Keystone_5005-5009_Compact" (at 129.54 109.22 0)
+    (property "Footprint" "TestPoint:TestPoint_Pad_2.0x2.0mm" (at 129.54 109.22 0)
       (effects (font (size 1.27 1.27)) hide)
     )
@@
       (effects (font (size 1.27 1.27)))
     )
-    (property "Footprint" "TestPoint:TestPoint_Keystone_5005-5009_Compact" (at 141.605 113.665 0)
+    (property "Footprint" "TestPoint:TestPoint_Pad_2.0x2.0mm" (at 141.605 113.665 0)
       (effects (font (size 1.27 1.27)) hide)
     )
@@
       (effects (font (size 1.27 1.27)))
     )
-    (property "Footprint" "My0R:RESC1005X40N" (at 240.03 103.505 0)
+    (property "Footprint" "Resistor_SMD:R_0402_1005Metric" (at 240.03 103.505 0)
       (effects (font (size 1.27 1.27)) (justify left) hide)
     )
@@
       (effects (font (size 1.27 1.27)) (justify left))
     )
-    (property "Footprint" "TestPoint:TestPoint_Keystone_5005-5009_Compact" (at 219.075 132.08 0)
+    (property "Footprint" "TestPoint:TestPoint_Pad_2.0x2.0mm" (at 219.075 132.08 0)
       (effects (font (size 1.27 1.27)) hide)
     )
@@
       (effects (font (size 1.27 1.27)))
     )
-    (property "Footprint" "My0R:RESC1005X40N" (at 160.655 117.475 0)
+    (property "Footprint" "Resistor_SMD:R_0402_1005Metric" (at 160.655 117.475 0)
       (effects (font (size 1.27 1.27)) (justify left) hide)
     )
@@
       (effects (font (size 1.27 1.27)))
     )
-    (property "Footprint" "My0R:RESC1005X40N" (at 129.54 41.275 0)
+    (property "Footprint" "Resistor_SMD:R_0402_1005Metric" (at 129.54 41.275 0)
       (effects (font (size 1.27 1.27)) (justify left) hide)
     )
@@
       (effects (font (size 1.27 1.27)) (justify left))
     )
-    (property "Footprint" "TestPoint:TestPoint_Keystone_5005-5009_Compact" (at 218.44 104.775 0)
+    (property "Footprint" "TestPoint:TestPoint_Pad_2.0x2.0mm" (at 218.44 104.775 0)
       (effects (font (size 1.27 1.27)) hide)
     )
@@
       (effects (font (size 1.27 1.27)))
     )
-    (property "Footprint" "My0R:RESC1005X40N" (at 69.215 107.95 0)
+    (property "Footprint" "Resistor_SMD:R_0402_1005Metric" (at 69.215 107.95 0)
       (effects (font (size 1.27 1.27)) (justify left) hide)
     )
@@
       (effects (font (size 1.27 1.27)) (justify left))
     )
-    (property "Footprint" "TestPoint:TestPoint_Keystone_5005-5009_Compact" (at 49.53 109.22 0)
-      (effects (font (size 1.27 1.27)) hide)
-    )
+    (property "Footprint" "TestPoint:TestPoint_Pad_2.0x2.0mm" (at 49.53 109.22 0)
+      (effects (font (size 1.27 1.27)) hide)
+    )
