File: EEE3088/Power_kicad_sch.kicad_sch (KiCad schematic)
At the start: 28 parts, among them U1 TP4056, U2 HT7533-1

Commit message: H_1
Parts:
- added TP12, TP14: TestPoint, TestPoint:TestPoint_Pad_2.0x2.0mm, symbol Connector:TestPoint
Connections:
- net +3.3V: now also TP5.1
- net +5V: now also TP14.1
- net GND: now also TP12.1; no longer Op-Amp1.5 (VINB+), Op-Amp1.6 (VINB-)
- net at R9.1, U2.3 (VO): no longer TP5.1
Other:
- moved on the sheet: BT1, C1, C2, LED1, LED2, N-Mos1, Op-Amp1, P-Mos1, R10, R2, R32, R4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

Commit message: Schematic updates
Parts:
- BT1: JLC Part Number (none) -> DNP; Manufacturer_Part_Number - -> DNP; Price 0.00 -> 0
- C1, C2: JLC Part Number C19702 -> C15850; Manufacturer_Part_Number CL10A106KP8NNNC -> CL21A106KAYNNNE; Price 0.0066 -> 0.0131
- N-Mos1: Price 0.0864 -> 0.0787
- Op-Amp1: Price 0.282 -> 0.2660
- P-Mos1: Price 0.0797 -> 0.0765
- R10, R4, R6, R8, R9: JLC Part Number C17168 -> C17477; Manufacturer_Part_Number 0402WGF0000TCE -> 0805W8F0000T5E; Price 0.0035 -> 0.0022
- R2: JLC Part Number C22765 -> C17379; Manufacturer_Part_Number 0603WAF1201T5E -> 0805W8F1201T5E; Price 0.001 -> 0.0018
- R32, R4: JLC Part Number C21190 -> C17513; Manufacturer_Part_Number 0603WAF1001T5E -> 0805W8F1001T5E; Price 0.0006 -> 0.0021
- R5: JLC Part Number C17900 -> C149504; Manufacturer_Part_Number 1206W4F1003T5E -> 0805W8F1003T5E; Price 0.0032 -> 0.0017
- TP1, TP12, TP14, TP2, TP3, TP4, TP5: JLC Part Number (none) -> DNP; Manufacturer_Part_Number 0 -> DNP
- TP22: Extended (none) -> 0; JLC Part Number (none) -> DNP; Manufacturer_Part_Number (none) -> DNP; Price (none) -> 0
- U1: Price 0.2064 -> 0.2121
- U2, Voltage-Regulator-1: Price 0.1315 -> 0.1279
- Z1: Manufacturer_Part_Number MM3Z5V6C -> MM3Z5V6; Price 0.0184 -> 0.0182

Commit message: Schematic + PCB Update
Parts:
- C1, C2: footprint CL10A106KP8NNNC:CAPC1608X90N -> Capacitor_SMD:C_0805_2012Metric
- R10, R4, R6, R8, R9: footprint Resistor_SMD:R_0402_1005Metric -> Resistor_SMD:R_0805_2012Metric
- R2: footprint My1.2k:RESC1608X55N -> Resistor_SMD:R_0805_2012Metric
- R32, R4: footprint RESC1608X55N -> Resistor_SMD:R_0805_2012Metric
- R5: footprint My100k:RESC3116X65N -> Resistor_SMD:R_0805_2012Metric
- R7: footprint My1M:RESC2013X65N -> Resistor_SMD:R_0805_2012Metric
Changed lines of the file:
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@@
       (effects (font (size 1.27 1.27)) (justify left))
     )
-    (property "Footprint" "My1M:RESC2013X65N" (at 148.59 158.115 0)
+    (property "Footprint" "Resistor_SMD:R_0805_2012Metric" (at 148.59 158.115 0)
       (effects (font (size 1.27 1.27)) (justify left) hide)
     )
@@
       (effects (font (size 1.27 1.27)) (justify right))
     )
-    (property "Footprint" "My100k:RESC3116X65N" (at 38.1 152.4 0)
+    (property "Footprint" "Resistor_SMD:R_0805_2012Metric" (at 38.1 152.4 0)
       (effects (font (size 1.27 1.27)) (justify left) hide)
     )
@@
       (effects (font (size 1.27 1.27)) (justify left))
     )
-    (property "Footprint" "RESC1608X55N" (at 113.03 49.53 0)
+    (property "Footprint" "Resistor_SMD:R_0805_2012Metric" (at 113.03 49.53 0)
       (effects (font (size 1.27 1.27)) (justify left) hide)
     )
@@
       (effects (font (size 1.27 1.27)) (justify left) hide)
     )
-    (property "Description" "1k Res 0805" (at 107.95 49.53 0)
+    (property "Description" "1k Resistor 0805" (at 107.95 49.53 0)
       (effects (font (size 1.27 1.27)) (justify left) hide)
     )
@@
       (effects (font (size 1.27 1.27)))
     )
-    (property "Footprint" "Resistor_SMD:R_0402_1005Metric" (at 253.365 136.525 0)
+    (property "Footprint" "Resistor_SMD:R_0805_2012Metric" (at 253.365 136.525 0)
       (effects (font (size 1.27 1.27)) (justify left) hide)
     )
@@
       (effects (font (size 1.27 1.27)) (justify left) hide)
     )
-    (property "Description" "0 Res 0805" (at 253.365 141.605 0)
+    (property "Description" "0 Resistor 0805" (at 253.365 141.605 0)
       (effects (font (size 1.27 1.27)) (justify left) hide)
     )
@@
       (effects (font (size 1.27 1.27)))
     )
-    (property "Footprint" "CL10A106KP8NNNC:CAPC1608X90N" (at 34.29 40.64 0)
+    (property "Footprint" "Capacitor_SMD:C_0805_2012Metric" (at 34.29 40.64 0)
       (effects (font (size 1.27 1.27)) (justify bottom) hide)
     )
@@
       (effects (font (size 1.27 1.27)))
     )
-    (property "Footprint" "Resistor_SMD:R_0402_1005Metric" (at 254 109.22 0)
+    (property "Footprint" "Resistor_SMD:R_0805_2012Metric" (at 254 109.22 0)
       (effects (font (size 1.27 1.27)) (justify left) hide)
     )
@@
       (effects (font (size 1.27 1.27)) (justify left) hide)
     )
-    (property "Description" "0 Res 0805" (at 254 114.3 0)
+    (property "Description" "0 Resistor 0805" (at 254 114.3 0)
       (effects (font (size 1.27 1.27)) (justify left) hide)
     )
@@
       (effects (font (size 1.27 1.27)))
     )
-    (property "Footprint" "Resistor_SMD:R_0402_1005Metric" (at 161.29 138.43 0)
+    (property "Footprint" "Resistor_SMD:R_0805_2012Metric" (at 161.29 138.43 0)
       (effects (font (size 1.27 1.27)) (justify left) hide)
     )
@@
       (effects (font (size 1.27 1.27)) (justify left) hide)
     )
-    (property "Description" "0 Res 0805" (at 161.29 143.51 0)
+    (property "Description" "0 Resistor 0805" (at 161.29 143.51 0)
       (effects (font (size 1.27 1.27)) (justify left) hide)
     )
@@
       (effects (font (size 1.27 1.27)) (justify right))
     )
-    (property "Footprint" "CL10A106KP8NNNC:CAPC1608X90N" (at 99.695 62.865 0)
+    (property "Footprint" "Capacitor_SMD:C_0805_2012Metric" (at 99.695 62.865 0)
       (effects (font (size 1.27 1.27)) (justify bottom) hide)
     )
@@
       (effects (font (size 1.27 1.27)))
     )
-    (property "Footprint" "Resistor_SMD:R_0402_1005Metric" (at 140.97 50.8 0)
+    (property "Footprint" "Resistor_SMD:R_0805_2012Metric" (at 140.97 50.8 0)
       (effects (font (size 1.27 1.27)) (justify left) hide)
     )
@@
       (effects (font (size 1.27 1.27)) (justify left) hide)
     )
-    (property "Description" "0 Res 0805" (at 140.97 55.88 0)
+    (property "Description" "0 Resistor 0805" (at 140.97 55.88 0)
       (effects (font (size 1.27 1.27)) (justify left) hide)
     )
@@
       (effects (font (size 1.27 1.27)))
     )
-    (property "Footprint" "Resistor_SMD:R_0402_1005Metric" (at 70.485 130.81 0)
+    (property "Footprint" "Resistor_SMD:R_0805_2012Metric" (at 70.485 130.81 0)
       (effects (font (size 1.27 1.27)) (justify left) hide)
     )
@@
       (effects (font (size 1.27 1.27)) (justify left) hide)
     )
-    (property "Description" "0 Res 0805" (at 70.485 135.89 0)
+    (property "Description" "0 Resistor 0805" (at 70.485 135.89 0)
       (effects (font (size 1.27 1.27)) (justify left) hide)
     )
@@
       (effects (font (size 1.27 1.27)) (justify right))
     )
-    (property "Footprint" "RESC1608X55N" (at 33.02 60.325 0)
+    (property "Footprint" "Resistor_SMD:R_0805_2012Metric" (at 33.02 60.325 0)
       (effects (font (size 1.27 1.27)) (justify left) hide)
     )
@@
       (effects (font (size 1.27 1.27)) (justify left) hide)
     )
-    (property "Description" "1k Res 0805" (at 38.1 60.325 0)
+    (property "Description" "1k Resistor 0805" (at 38.1 60.325 0)
       (effects (font (size 1.27 1.27)) (justify left) hide)
     )
@@
       (effects (font (size 1.27 1.27)))
     )
-    (property "Footprint" "My1.2k:RESC1608X55N" (at 43.815 67.945 0)
-      (effects (font (size 1.27 1.27)) (justify left) hide)
-    )
+    (property "Footprint" "Resistor_SMD:R_0805_2012Metric" (at 43.815 67.945 0)
+      (effects (font (size 1.27 1.27)) (justify left) hide)
+    )

Commit message: PCB continued again
Parts:
- renumbered R32 to R1, R8 to R7, R7 to R8, TP12 to TP2, TP14 to TP3, TP2 to TP4, TP22 to TP5, TP3 to TP6, TP4 to TP7, TP5 to TP8, Voltage-Regulator-1 to U1, Op-Amp1 to U9

Commit message: PCD- stm header added
Parts:
- U1, U2: footprint HT7533-1:SOT89 -> Package_TO_SOT_SMD:SOT-89-3
- U1: footprint TP4056:SOP127P600X175-9N -> Package_SO:SOP-8-1EP_4.57x4.57mm_P1.27mm_EP4.57x4.45mm
- U9: footprint Myopamp:SOIC127P600X175-8N -> Package_SO:SOIC-8-1EP_3.9x4.9mm_P1.27mm_EP2.29x3mm
Connections:
- net GND: now also U9.5 (VINB+), U9.6 (VINB-)
Changed lines of the file:
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@@
   (junction (at 52.07 50.165) (diameter 0) (color 0 0 0 0)
+  )
+  (junction (at 94.615 139.7) (diameter 0) (color 0 0 0 0)
   )
   (junction (at 147.32 139.7) (diameter 0) (color 0 0 0 0)
@@
     (stroke (width 0) (type default))
   )
-  (wire (pts (xy 98.425 133.35) (xy 98.425 136.525))
+  (wire (pts (xy 94.615 137.16) (xy 94.615 139.7))
     (stroke (width 0) (type default))
   )
@@
   )
   (wire (pts (xy 52.07 34.29) (xy 66.675 34.29))
+    (stroke (width 0) (type default))
+  )
+  (wire (pts (xy 94.615 139.7) (xy 94.615 140.335))
     (stroke (width 0) (type default))
   )
@@
       (effects (font (size 1.27 1.27)))
     )
-    (property "Footprint" "HT7533-1:SOT89" (at 207.645 113.03 0)
+    (property "Footprint" "Package_TO_SOT_SMD:SOT-89-3" (at 207.645 113.03 0)
       (effects (font (size 1.27 1.27)) (justify bottom) hide)
     )
@@
       (effects (font (size 1.27 1.27)))
     )
-    (property "Footprint" "HT7533-1:SOT89" (at 207.645 140.335 0)
+    (property "Footprint" "Package_TO_SOT_SMD:SOT-89-3" (at 207.645 140.335 0)
       (effects (font (size 1.27 1.27)) (justify bottom) hide)
     )
@@
       (effects (font (size 1.27 1.27)))
     )
-    (property "Footprint" "TP4056:SOP127P600X175-9N" (at 78.105 57.15 0)
+    (property "Footprint" "Package_SO:SOP-8-1EP_4.57x4.57mm_P1.27mm_EP4.57x4.45mm" (at 78.105 57.15 0)
       (effects (font (size 1.27 1.27)) (justify bottom) hide)
     )
@@
       (effects (font (size 1.27 1.27)) (justify left))
     )
-    (property "Footprint" "Myopamp:SOIC127P600X175-8N" (at 124.46 121.92 0)
-      (effects (font (size 1.27 1.27)) (justify left) hide)
-    )
+    (property "Footprint" "Package_SO:SOIC-8-1EP_3.9x4.9mm_P1.27mm_EP2.29x3mm" (at 124.46 121.92 0)
+      (effects (font (size 1.27 1.27)) (justify left) hide)
+    )

Commit message: PCB-Final
Parts:
- renumbered N-Mos1 to N1, P-Mos1 to P1
Changed lines of the file:
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@@
     (stroke (width 0) (type default))
   )
-  (wire (pts (xy 259.08 137.795) (xy 260.985 137.795))
+  (wire (pts (xy 259.08 137.795) (xy 273.05 137.795))
     (stroke (width 0) (type default))
   )
@@
     (effects (font (size 1.27 1.27)) (justify left bottom))
   )
-  (global_label "+3.3V" (shape output) (at 260.985 137.795 0) (fields_autoplaced)
-    (effects (font (size 1.27 1.27)) (justify left))
-    (property "Intersheetrefs" "${INTERSHEET_REFS}" (at 269.5756 137.795 0)
-      (effects (font (size 1.27 1.27)) (justify left) hide)
-    )
-  )
   (symbol (lib_id "power:GND") (at 207.645 118.11 0) (unit 1)
     (in_bom yes) (on_board yes) (dnp no) (fields_autoplaced)
@@
   (symbol (lib_id "AO3400A:AO3400A") (at 139.7 132.08 0) (unit 1)
     (in_bom yes) (on_board yes) (dnp no) (fields_autoplaced)
-    (property "Reference" "N-Mos1" (at 151.13 128.905 0)
+    (property "Reference" "N1" (at 151.13 128.905 0)
       (effects (font (size 1.27 1.27)) (justify left))
     )
@@
       (project "EEE3088"
         (path "/83bdd5e1-981a-4ca1-9a2f-70dea9f00850/1213f935-6f8d-4a20-9c2e-6b5e9a834fe6"
-          (reference "N-Mos1") (unit 1)
+          (reference "N1") (unit 1)
         )
       )
@@
         (path "/83bdd5e1-981a-4ca1-9a2f-70dea9f00850/1213f935-6f8d-4a20-9c2e-6b5e9a834fe6"
           (reference "R9") (unit 1)
+        )
+      )
+    )
+  )
+  (symbol (lib_id "power:+3.3V") (at 273.05 137.795 0) (unit 1)
+    (in_bom yes) (on_board yes) (dnp no) (fields_autoplaced)
+    (property "Reference" "#PWR044" (at 273.05 141.605 0)
+      (effects (font (size 1.27 1.27)) hide)
+    )
+    (property "Value" "+3.3V" (at 273.05 133.985 0)
+      (effects (font (size 1.27 1.27)))
+    )
+    (property "Footprint" "" (at 273.05 137.795 0)
+      (effects (font (size 1.27 1.27)) hide)
+    )
+    (property "Datasheet" "" (at 273.05 137.795 0)
+      (effects (font (size 1.27 1.27)) hide)
+    )
+    (pin "1")
+    (instances
+      (project "EEE3088"
+        (path "/83bdd5e1-981a-4ca1-9a2f-70dea9f00850/d16a673b-d677-4a4a-a11c-ee22bd422692"
+          (reference "#PWR044") (unit 1)
+        )
+        (path "/83bdd5e1-981a-4ca1-9a2f-70dea9f00850"
+          (reference "#PWR01") (unit 1)
+        )
+        (path "/83bdd5e1-981a-4ca1-9a2f-70dea9f00850/1213f935-6f8d-4a20-9c2e-6b5e9a834fe6"
+          (reference "#PWR01") (unit 1)
         )
       )
@@
   (symbol (lib_id "AO3401A:AO3401A") (at 39.37 139.7 90) (unit 1)
     (in_bom yes) (on_board yes) (dnp no) (fields_autoplaced)
-    (property "Reference" "P-Mos1" (at 36.83 125.73 90)
+    (property "Reference" "P1" (at 36.83 125.73 90)
       (effects (font (size 1.27 1.27)))
     )
@@
       (project "EEE3088"
         (path "/83bdd5e1-981a-4ca1-9a2f-70dea9f00850/1213f935-6f8d-4a20-9c2e-6b5e9a834fe6"
-          (reference "P-Mos1") (unit 1)
-        )
-      )
+          (reference "P1") (unit 1)
+        )
+      )

Commit message: Update Power_kicad_sch.kicad_sch
Connections:
- net GND: now also BT1.N
- net V-Reg: no longer U1.2 (VI), U1.2@1 (VI)
- net V-pos: now also U1.2 (VI), U1.2@1 (VI)
- net Vbat: now also BT1.P, P1.3; no longer BT1.N
Other:
- moved on the sheet: BT1
Changed lines of the file:
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@@
   (junction (at 52.07 50.165) (diameter 0) (color 0 0 0 0)
+  )
+  (junction (at 33.02 116.205) (diameter 0) (color 0 0 0 0)
   )
   (junction (at 94.615 139.7) (diameter 0) (color 0 0 0 0)
@@
     (stroke (width 0) (type default))
   )
+  (wire (pts (xy 56.515 110.49) (xy 56.515 116.205))
+    (stroke (width 0) (type default))
+  )
   (wire (pts (xy 190.5 110.49) (xy 197.485 110.49))
     (stroke (width 0) (type default))
@@
     (stroke (width 0) (type default))
   )
+  (wire (pts (xy 33.02 116.205) (xy 33.02 123.19))
+    (stroke (width 0) (type default))
+  )
   (wire (pts (xy 29.21 123.19) (xy 29.21 132.08))
     (stroke (width 0) (type default))
@@
     (stroke (width 0) (type default))
   )
+  (wire (pts (xy 56.515 116.205) (xy 33.02 116.205))
+    (stroke (width 0) (type default))
+  )
   (wire (pts (xy 52.07 34.29) (xy 34.29 34.29))
     (stroke (width 0) (type default))
@@
     (stroke (width 0) (type default))
   )
+  (wire (pts (xy 33.02 123.19) (xy 29.21 123.19))
+    (stroke (width 0) (type default))
+  )
   (wire (pts (xy 49.53 132.08) (xy 49.53 133.35))
-    (stroke (width 0) (type default))
-  )
-  (wire (pts (xy 56.515 110.49) (xy 29.21 110.49))
     (stroke (width 0) (type default))
   )
@@
     (effects (font (size 1.27 1.27)) (justify left bottom))
   )
-  (label "V-Reg" (at 190.5 110.49 0) (fields_autoplaced)
+  (label "V-pos" (at 190.5 110.49 0) (fields_autoplaced)
     (effects (font (size 1.27 1.27)) (justify left bottom))
   )
@@
     )
   )
-  (symbol (lib_id "BH-18650-PC:BH-18650-PC") (at 29.21 115.57 90) (unit 1)
-    (in_bom yes) (on_board yes) (dnp no) (fields_autoplaced)
-    (property "Reference" "BT1" (at 33.02 117.475 90)
-      (effects (font (size 1.27 1.27)) (justify right))
-    )
-    (property "Value" "BH-18650-PC" (at 33.02 120.015 90)
-      (effects (font (size 1.27 1.27)) (justify right))
-    )
-    (property "Footprint" "BH-18650-PC:BAT_BH-18650-PC" (at 29.21 115.57 0)
+  (symbol (lib_id "BH-18650-PC:BH-18650-PC") (at 25.4 116.205 180) (unit 1)
+    (in_bom yes) (on_board yes) (dnp no) (fields_autoplaced)
+    (property "Reference" "BT1" (at 27.94 109.855 0)
+      (effects (font (size 1.27 1.27)))
+    )
+    (property "Value" "BH-18650-PC" (at 27.94 112.395 0)
+      (effects (font (size 1.27 1.27)))
+    )
+    (property "Footprint" "BH-18650-PC:BAT_BH-18650-PC" (at 25.4 116.205 0)
       (effects (font (size 1.27 1.27)) (justify bottom) hide)
     )
-    (property "Datasheet" "-" (at 29.21 115.57 0)
-      (effects (font (size 1.27 1.27)) hide)
-    )
-    (property "MANUFACTURER" "MPD" (at 29.21 115.57 0)
+    (property "Datasheet" "-" (at 25.4 116.205 0)
+      (effects (font (size 1.27 1.27)) hide)
+    )
+    (property "MANUFACTURER" "MPD" (at 25.4 116.205 0)
       (effects (font (size 1.27 1.27)) (justify bottom) hide)
     )
-    (property "STANDARD" "Manufacturer Recommendation" (at 29.21 115.57 0)
+    (property "STANDARD" "Manufacturer Recommendation" (at 25.4 116.205 0)
       (effects (font (size 1.27 1.27)) (justify bottom) hide)
     )
-    (property "PARTREV" "05/17/19" (at 29.21 115.57 0)
+    (property "PARTREV" "05/17/19" (at 25.4 116.205 0)
       (effects (font (size 1.27 1.27)) (justify bottom) hide)
     )
-    (property "MAXIMUM_PACKAGE_HEIGHT" "21.31mm" (at 29.21 115.57 0)
+    (property "MAXIMUM_PACKAGE_HEIGHT" "21.31mm" (at 25.4 116.205 0)
       (effects (font (size 1.27 1.27)) (justify bottom) hide)
     )
-    (property "Price" "0" (at 29.21 115.57 0)
-      (effects (font (size 1.27 1.27)) hide)
-    )
-    (property "Basic" "" (at 29.21 115.57 0)
-      (effects (font (size 1.27 1.27)) hide)
-    )
-    (property "Extended" "0" (at 29.21 115.57 0)
-      (effects (font (size 1.27 1.27)) hide)
-    )
-    (property "Description" "Battery Holder" (at 29.21 115.57 0)
-      (effects (font (size 1.27 1.27)) hide)
-    )
-    (property "Manufacturer_Part_Number" "DNP" (at 29.21 115.57 0)
-      (effects (font (size 1.27 1.27)) hide)
-    )
-    (property "JLC Part Number" "DNP" (at 29.21 115.57 0)
+    (property "Price" "0" (at 25.4 116.205 0)
+      (effects (font (size 1.27 1.27)) hide)
+    )
+    (property "Basic" "" (at 25.4 116.205 0)
+      (effects (font (size 1.27 1.27)) hide)
+    )
+    (property "Extended" "0" (at 25.4 116.205 0)
+      (effects (font (size 1.27 1.27)) hide)
+    )
+    (property "Description" "Battery Holder" (at 25.4 116.205 0)
+      (effects (font (size 1.27 1.27)) hide)
+    )
+    (property "Manufacturer_Part_Number" "DNP" (at 25.4 116.205 0)
+      (effects (font (size 1.27 1.27)) hide)
+    )
+    (property "JLC Part Number" "DNP" (at 25.4 116.205 0)
       (effects (font (size 1.27 1.27)) hide)
     )
@@
         )
       )
+    )
+  )
+  (symbol (lib_id "power:GND") (at 20.32 116.205 0) (unit 1)
+    (in_bom yes) (on_board yes) (dnp no) (fields_autoplaced)
+    (property "Reference" "#PWR046" (at 20.32 122.555 0)
+      (effects (font (size 1.27 1.27)) hide)
+    )
+    (property "Value" "GND" (at 20.32 120.65 0)
+      (effects (font (size 1.27 1.27)))
+    )
+    (property "Footprint" "" (at 20.32 116.205 0)
+      (effects (font (size 1.27 1.27)) hide)
+    )
+    (property "Datasheet" "" (at 20.32 116.205 0)
+      (effects (font (size 1.27 1.27)) hide)
+    )
+    (pin "1")
+    (instances
+      (project "EEE3088"
+        (path "/83bdd5e1-981a-4ca1-9a2f-70dea9f00850/1213f935-6f8d-4a20-9c2e-6b5e9a834fe6"
+          (reference "#PWR046") (unit 1)
+        )
+      )
