File: EEE3088/Microcontroller_kicad_sch.kicad_sch (KiCad schematic)
At the start: 12 parts, among them J2 Conn_01x24, J3 Conn_01x24

Commit message: updated BOM
Parts:
- C?: footprint CL21B105KBFNNNE -> (none)
- C? (x2): Extended (none) -> 0; Manufacturer_Part_Number (none) -> CC0603KRX7R9BB104; Price (none) -> 0.01
- C?: Extended (none) -> 0; Manufacturer_Part_Number (none) -> CL21A475KAQNNNE; Price (none) -> 0.01
- C?: footprint (none) -> CL21B103KBANNNC; Extended (none) -> 0; Manufacturer_Part_Number (none) -> CL21B103KBANNNC; Price (none) -> 0.01
- J?: Extended (none) -> 0; Manufacturer_Part_Number (none) -> MicroXNJ; Price (none) -> 0.03
- U?: Extended (none) -> 0; Manufacturer_Part_Number (none) -> AT24C256C-SSHL-T
- U?: Extended (none) -> 0; Manufacturer_Part_Number (none) -> CH340G; Price (none) -> 0.47
Changed lines of the file:
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@@
       (effects (font (size 1.27 1.27)) (justify left))
     )
-    (property "Footprint" "CL21B105KBFNNNE" (at 247.8532 96.012 0)
+    (property "Footprint" "" (at 247.8532 96.012 0)
       (effects (font (size 1.27 1.27)) hide)
     )
@@
       (effects (font (size 1.27 1.27)) (justify bottom) hide)
     )
-    (property "Datasheet" "" (at 160.02 49.022 0)
+    (property "Datasheet" "https://datasheet.lcsc.com/lcsc/1809151932_Microchip-Tech-AT24C256C-SSHL-T_C6482.pdf" (at 160.02 49.022 0)
       (effects (font (size 1.27 1.27)) hide)
     )
@@
       (effects (font (size 1.27 1.27)) hide)
     )
-    (property "Extended" "" (at 160.02 49.022 0)
+    (property "Extended" "0" (at 160.02 49.022 0)
+      (effects (font (size 1.27 1.27)) hide)
+    )
+    (property "Manufacturer_Part_Number" "AT24C256C-SSHL-T" (at 160.02 49.022 0)
       (effects (font (size 1.27 1.27)) hide)
     )
@@
       (effects (font (size 1.27 1.27)) (justify bottom) hide)
     )
-    (property "Datasheet" "" (at 251.714 46.482 0)
+    (property "Datasheet" "https://datasheet.lcsc.com/lcsc/2008191806_WCH-Jiangsu-Qin-Heng-CH340G_C14267.pdf" (at 251.714 46.482 0)
       (effects (font (size 1.27 1.27)) hide)
     )
@@
       (effects (font (size 1.27 1.27)) (justify bottom) hide)
     )
-    (property "Price" "" (at 251.714 46.482 0)
+    (property "Price" "0.47" (at 251.714 46.482 0)
       (effects (font (size 1.27 1.27)) hide)
     )
@@
       (effects (font (size 1.27 1.27)) hide)
     )
-    (property "Extended" "" (at 251.714 46.482 0)
+    (property "Extended" "0" (at 251.714 46.482 0)
+      (effects (font (size 1.27 1.27)) hide)
+    )
+    (property "Manufacturer_Part_Number" "CH340G" (at 251.714 46.482 0)
       (effects (font (size 1.27 1.27)) hide)
     )
@@
       (effects (font (size 1.27 1.27)) (justify bottom) hide)
     )
-    (property "Datasheet" "" (at 38.354 40.894 0)
+    (property "Datasheet" "https://datasheet.lcsc.com/lcsc/2204151400_SHOU-HAN-MicroXNJ_C404969.pdf" (at 38.354 40.894 0)
       (effects (font (size 1.27 1.27)) hide)
     )
@@
       (effects (font (size 1.27 1.27)) (justify bottom) hide)
     )
-    (property "Price" "" (at 38.354 40.894 0)
+    (property "Price" "0.03" (at 38.354 40.894 0)
       (effects (font (size 1.27 1.27)) hide)
     )
@@
       (effects (font (size 1.27 1.27)) hide)
     )
-    (property "Extended" "" (at 38.354 40.894 0)
+    (property "Extended" "0" (at 38.354 40.894 0)
+      (effects (font (size 1.27 1.27)) hide)
+    )
+    (property "Description" "USB interface" (at 38.354 40.894 0)
+      (effects (font (size 1.27 1.27)) hide)
+    )
+    (property "Manufacturer_Part_Number" "MicroXNJ" (at 38.354 40.894 0)
       (effects (font (size 1.27 1.27)) hide)
     )
@@
       (effects (font (size 1.27 1.27)) hide)
     )
-    (property "Datasheet" "~" (at 203.708 92.202 0)
-      (effects (font (size 1.27 1.27)) hide)
-    )
-    (property "Price" "" (at 203.708 92.202 0)
+    (property "Datasheet" "https://datasheet.lcsc.com/lcsc/2211101700_YAGEO-CC0603KRX7R9BB104_C14663.pdf" (at 203.708 92.202 0)
+      (effects (font (size 1.27 1.27)) hide)
+    )
+    (property "Price" "0.01" (at 203.708 92.202 0)
       (effects (font (size 1.27 1.27)) hide)
     )
@@
       (effects (font (size 1.27 1.27)) hide)
     )
-    (property "Extended" "" (at 203.708 92.202 0)
+    (property "Extended" "0" (at 203.708 92.202 0)
+      (effects (font (size 1.27 1.27)) hide)
+    )
+    (property "Description" "100nF Cap" (at 203.708 92.202 0)
+      (effects (font (size 1.27 1.27)) hide)
+    )
+    (property "Manufacturer_Part_Number" "CC0603KRX7R9BB104" (at 203.708 92.202 0)
       (effects (font (size 1.27 1.27)) hide)
     )
@@
       (effects (font (size 1.27 1.27)) hide)
     )
-    (property "Datasheet" "~" (at 222.758 92.202 0)
-      (effects (font (size 1.27 1.27)) hide)
-    )
-    (property "Price" "" (at 222.758 92.202 0)
+    (property "Datasheet" "https://datasheet.lcsc.com/lcsc/1810261822_Samsung-Electro-Mechanics-CL21A475KAQNNNE_C1779.pdf" (at 222.758 92.202 0)
+      (effects (font (size 1.27 1.27)) hide)
+    )
+    (property "Price" "0.01" (at 222.758 92.202 0)
       (effects (font (size 1.27 1.27)) hide)
     )
@@
       (effects (font (size 1.27 1.27)) hide)
     )
-    (property "Extended" "" (at 222.758 92.202 0)
+    (property "Extended" "0" (at 222.758 92.202 0)
+      (effects (font (size 1.27 1.27)) hide)
+    )
+    (property "Description" "4.7uF" (at 222.758 92.202 0)
+      (effects (font (size 1.27 1.27)) hide)
+    )
+    (property "Manufacturer_Part_Number" "CL21A475KAQNNNE" (at 222.758 92.202 0)
       (effects (font (size 1.27 1.27)) hide)
     )
@@
       (effects (font (size 1.27 1.27)) (justify left))
     )
-    (property "Footprint" "" (at 237.6932 96.012 0)
-      (effects (font (size 1.27 1.27)) hide)
-    )
-    (property "Datasheet" "~" (at 236.728 92.202 0)
-      (effects (font (size 1.27 1.27)) hide)
-    )
-    (property "Price" "" (at 236.728 92.202 0)
+    (property "Footprint" "CL21B103KBANNNC" (at 237.6932 96.012 0)
+      (effects (font (size 1.27 1.27)) hide)
+    )
+    (property "Datasheet" "https://datasheet.lcsc.com/lcsc/1811151136_Samsung-Electro-Mechanics-CL21B103KBANNNC_C1710.pdf" (at 236.728 92.202 0)
+      (effects (font (size 1.27 1.27)) hide)
+    )
+    (property "Price" "0.01" (at 236.728 92.202 0)
       (effects (font (size 1.27 1.27)) hide)
     )
@@
       (effects (font (size 1.27 1.27)) hide)
     )
-    (property "Extended" "" (at 236.728 92.202 0)
+    (property "Extended" "0" (at 236.728 92.202 0)
+      (effects (font (size 1.27 1.27)) hide)
+    )
+    (property "Description" "10nF Cap" (at 236.728 92.202 0)
+      (effects (font (size 1.27 1.27)) hide)
+    )
+    (property "Manufacturer_Part_Number" "CL21B103KBANNNC" (at 236.728 92.202 0)
       (effects (font (size 1.27 1.27)) hide)
     )
@@
       (effects (font (size 1.27 1.27)) hide)
     )
-    (property "Datasheet" "~" (at 213.868 92.202 0)
-      (effects (font (size 1.27 1.27)) hide)
-    )
-    (property "Price" "" (at 213.868 92.202 0)
+    (property "Datasheet" "https://datasheet.lcsc.com/lcsc/2211101700_YAGEO-CC0603KRX7R9BB104_C14663.pdf" (at 213.868 92.202 0)
+      (effects (font (size 1.27 1.27)) hide)
+    )
+    (property "Price" "0.01" (at 213.868 92.202 0)
       (effects (font (size 1.27 1.27)) hide)
     )
@@
       (effects (font (size 1.27 1.27)) hide)
     )
-    (property "Extended" "" (at 213.868 92.202 0)
-      (effects (font (size 1.27 1.27)) hide)
-    )
+    (property "Extended" "0" (at 213.868 92.202 0)
+      (effects (font (size 1.27 1.27)) hide)
+    )
+    (property "Description" "100nF Cap" (at 213.868 92.202 0)
+      (effects (font (size 1.27 1.27)) hide)
+    )
+    (property "Manufacturer_Part_Number" "CC0603KRX7R9BB104" (at 213.868 92.202 0)
+      (effects (font (size 1.27 1.27)) hide)
+    )

Commit message: BOM attempt
Parts:
- C?: Manufacturer_Part_Number (none) -> -
- J2, J3: Extended (none) -> -; Manufacturer_Part_Number (none) -> -; Price (none) -> -
- U?: Price (none) -> 0.5313
Changed lines of the file:
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@@
+      (effects (font (size 1.27 1.27)) hide)
+    )
+    (property "Manufacturer_Part_Number" "-" (at 246.888 92.202 0)
       (effects (font (size 1.27 1.27)) hide)
     )
@@
       (effects (font (size 1.27 1.27)) (justify bottom) hide)
     )
-    (property "Price" "" (at 160.02 49.022 0)
+    (property "Price" "0.5313" (at 160.02 49.022 0)
       (effects (font (size 1.27 1.27)) hide)
     )
@@
       (effects (font (size 1.27 1.27)) hide)
     )
-    (property "Description" "USB interface" (at 38.354 40.894 0)
+    (property "Description" "-" (at 38.354 40.894 0)
       (effects (font (size 1.27 1.27)) hide)
     )
@@
       (effects (font (size 1.27 1.27)) hide)
     )
-    (property "Datasheet" "~" (at 83.058 60.198 0)
+    (property "Datasheet" "-" (at 83.058 60.198 0)
+      (effects (font (size 1.27 1.27)) hide)
+    )
+    (property "Description" "-" (at 83.058 60.198 0)
+      (effects (font (size 1.27 1.27)) hide)
+    )
+    (property "Extended" "-" (at 83.058 60.198 0)
+      (effects (font (size 1.27 1.27)) hide)
+    )
+    (property "Manufacturer_Part_Number" "-" (at 83.058 60.198 0)
+      (effects (font (size 1.27 1.27)) hide)
+    )
+    (property "Price" "-" (at 83.058 60.198 0)
       (effects (font (size 1.27 1.27)) hide)
     )
@@
       (effects (font (size 1.27 1.27)) hide)
     )
-    (property "Datasheet" "~" (at 108.458 60.452 0)
-      (effects (font (size 1.27 1.27)) hide)
-    )
+    (property "Datasheet" "-" (at 108.458 60.452 0)
+      (effects (font (size 1.27 1.27)) hide)
+    )
+    (property "Description" "-" (at 108.458 60.452 0)
+      (effects (font (size 1.27 1.27)) hide)
+    )
+    (property "Extended" "-" (at 108.458 60.452 0)
+      (effects (font (size 1.27 1.27)) hide)
+    )
+    (property "Manufacturer_Part_Number" "-" (at 108.458 60.452 0)
+      (effects (font (size 1.27 1.27)) hide)
+    )
+    (property "Price" "-" (at 108.458 60.452 0)
+      (effects (font (size 1.27 1.27)) hide)
+    )

Commit message: BOM Update
Parts:
- J2, J3: Extended - -> 0
Other:
- title: (none) -> MCU Schematic
Changed lines of the file:
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@@
   (paper "A4")
   (title_block
+    (title "MCU Schematic")
+    (date "2023-03-14")
+    (rev "Rev 1")
     (company "UCT")
+    (comment 1 "EEE3088F Project")
+    (comment 2 "Jack Youens")
   )
   (junction (at 73.66 32.258) (diameter 0) (color 0 0 0 0)
@@
     (fill (type none))
   )
+  (rectangle (start 166.37 77.47) (end 265.43 111.76)
+    (stroke (width 0) (type default))
+    (fill (type none))
+  )
   (rectangle (start 141.478 17.272) (end 215.392 65.786)
     (stroke (width 0) (type default))
@@
   )
   (symbol (lib_id "Device:C") (at 246.888 92.202 0) (unit 1)
-    (in_bom yes) (on_board yes) (dnp no) (fields_autoplaced)
-    (property "Reference" "C?" (at 250.698 91.567 0)
-      (effects (font (size 1.27 1.27)) (justify left))
-    )
-    (property "Value" "1uF" (at 250.698 94.107 0)
+    (in_bom yes) (on_board yes) (dnp no)
+    (property "Reference" "C?" (at 247.65 88.9 0)
+      (effects (font (size 1.27 1.27)) (justify left))
+    )
+    (property "Value" "1uF" (at 248.92 95.25 0)
       (effects (font (size 1.27 1.27)) (justify left))
     )
@@
     )
     (property "Manufacturer_Part_Number" "AT24C256C-SSHL-T" (at 160.02 49.022 0)
+      (effects (font (size 1.27 1.27)) hide)
+    )
+    (property "Description" "EEPROM" (at 160.02 49.022 0)
       (effects (font (size 1.27 1.27)) hide)
     )
@@
     )
     (property "Manufacturer_Part_Number" "CH340G" (at 251.714 46.482 0)
+      (effects (font (size 1.27 1.27)) hide)
+    )
+    (property "Description" "USB Comms IC" (at 251.714 46.482 0)
       (effects (font (size 1.27 1.27)) hide)
     )
@@
       (effects (font (size 1.27 1.27)) hide)
     )
-    (property "Description" "-" (at 38.354 40.894 0)
+    (property "Description" "Jumper" (at 38.354 40.894 0)
       (effects (font (size 1.27 1.27)) hide)
     )
@@
   )
   (symbol (lib_id "Device:C") (at 203.708 92.202 0) (unit 1)
-    (in_bom yes) (on_board yes) (dnp no) (fields_autoplaced)
-    (property "Reference" "C?" (at 207.518 91.567 0)
-      (effects (font (size 1.27 1.27)) (justify left))
-    )
-    (property "Value" "100nF" (at 207.518 94.107 0)
+    (in_bom yes) (on_board yes) (dnp no)
+    (property "Reference" "C?" (at 204.47 88.9 0)
+      (effects (font (size 1.27 1.27)) (justify left))
+    )
+    (property "Value" "100nF" (at 204.47 95.25 0)
       (effects (font (size 1.27 1.27)) (justify left))
     )
@@
       (effects (font (size 1.27 1.27)) (justify left) hide)
     )
-    (property "Description" "1K Resistor - 0402" (at 184.404 44.196 0)
+    (property "Description" "1k Resistor - 0805" (at 184.404 44.196 0)
       (effects (font (size 1.27 1.27)) (justify left) hide)
     )
@@
   )
   (symbol (lib_id "Device:C") (at 222.758 92.202 0) (unit 1)
-    (in_bom yes) (on_board yes) (dnp no) (fields_autoplaced)
-    (property "Reference" "C?" (at 226.568 91.567 0)
-      (effects (font (size 1.27 1.27)) (justify left))
-    )
-    (property "Value" "4.7uF" (at 226.568 94.107 0)
+    (in_bom yes) (on_board yes) (dnp no)
+    (property "Reference" "C?" (at 223.52 88.9 0)
+      (effects (font (size 1.27 1.27)) (justify left))
+    )
+    (property "Value" "4.7uF" (at 223.52 95.25 0)
       (effects (font (size 1.27 1.27)) (justify left))
     )
@@
       (effects (font (size 1.27 1.27)) hide)
     )
-    (property "Description" "-" (at 83.058 60.198 0)
-      (effects (font (size 1.27 1.27)) hide)
-    )
-    (property "Extended" "-" (at 83.058 60.198 0)
+    (property "Description" "STM Connector" (at 83.058 60.198 0)
+      (effects (font (size 1.27 1.27)) hide)
+    )
+    (property "Extended" "0" (at 83.058 60.198 0)
       (effects (font (size 1.27 1.27)) hide)
     )
@@
   )
   (symbol (lib_id "Device:C") (at 236.728 92.202 0) (unit 1)
-    (in_bom yes) (on_board yes) (dnp no) (fields_autoplaced)
-    (property "Reference" "C?" (at 240.538 91.567 0)
-      (effects (font (size 1.27 1.27)) (justify left))
-    )
-    (property "Value" "10nF" (at 240.538 94.107 0)
+    (in_bom yes) (on_board yes) (dnp no)
+    (property "Reference" "C?" (at 237.49 88.9 0)
+      (effects (font (size 1.27 1.27)) (justify left))
+    )
+    (property "Value" "10nF" (at 237.49 95.25 0)
       (effects (font (size 1.27 1.27)) (justify left))
     )
@@
       (effects (font (size 1.27 1.27)) hide)
     )
-    (property "Description" "-" (at 108.458 60.452 0)
-      (effects (font (size 1.27 1.27)) hide)
-    )
-    (property "Extended" "-" (at 108.458 60.452 0)
+    (property "Description" "STM Connector" (at 108.458 60.452 0)
+      (effects (font (size 1.27 1.27)) hide)
+    )
+    (property "Extended" "0" (at 108.458 60.452 0)
       (effects (font (size 1.27 1.27)) hide)
     )
@@
   )
   (symbol (lib_id "Device:C") (at 213.868 92.202 0) (unit 1)
-    (in_bom yes) (on_board yes) (dnp no) (fields_autoplaced)
-    (property "Reference" "C?" (at 217.678 91.567 0)
-      (effects (font (size 1.27 1.27)) (justify left))
-    )
-    (property "Value" "100nF" (at 217.678 94.107 0)
+    (in_bom yes) (on_board yes) (dnp no)
+    (property "Reference" "C?" (at 214.63 88.9 0)
+      (effects (font (size 1.27 1.27)) (justify left))
+    )
+    (property "Value" "100nF" (at 215.9 95.25 0)
       (effects (font (size 1.27 1.27)) (justify left))
     )
@@
       (effects (font (size 1.27 1.27)) (justify left) hide)
     )
-    (property "Description" "1K Resistor - 0402" (at 176.784 42.164 0)
-      (effects (font (size 1.27 1.27)) (justify left) hide)
-    )
+    (property "Description" "1k Resistor - 0805" (at 176.784 42.164 0)
+      (effects (font (size 1.27 1.27)) (justify left) hide)
+    )

Commit message: BOM_V1_Final
Parts:
- C? (x2): JLC Part Number (none) -> C14663
- C?: JLC Part Number (none) -> C1779
- C?: JLC Part Number (none) -> C1710
- R4: JLC Part Number (none) -> C17398; Manufacturer_Part_Number 0402WGF1001TCE -> 0805W8F1801T5E; Price 0.0005 -> 0.0018
- U?: JLC Part Number (none) -> C6482
- U?: JLC Part Number (none) -> C14267
Changed lines of the file:
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@@
+      (effects (font (size 1.27 1.27)) hide)
+    )
+    (property "JLC Part Number" "" (at 246.888 92.202 0)
       (effects (font (size 1.27 1.27)) hide)
     )
@@
     )
     (property "Description" "EEPROM" (at 160.02 49.022 0)
+      (effects (font (size 1.27 1.27)) hide)
+    )
+    (property "JLC Part Number" "C6482" (at 160.02 49.022 0)
       (effects (font (size 1.27 1.27)) hide)
     )
@@
     )
     (property "Description" "USB Comms IC" (at 251.714 46.482 0)
+      (effects (font (size 1.27 1.27)) hide)
+    )
+    (property "JLC Part Number" "C14267" (at 251.714 46.482 0)
       (effects (font (size 1.27 1.27)) hide)
     )
@@
     )
     (property "Manufacturer_Part_Number" "MicroXNJ" (at 38.354 40.894 0)
+      (effects (font (size 1.27 1.27)) hide)
+    )
+    (property "JLC Part Number" "" (at 38.354 40.894 0)
       (effects (font (size 1.27 1.27)) hide)
     )
@@
       (effects (font (size 1.27 1.27)) hide)
     )
+    (property "JLC Part Number" "C14663" (at 203.708 92.202 0)
+      (effects (font (size 1.27 1.27)) hide)
+    )
     (pin "1")
     (pin "2")
@@
       (effects (font (size 1.27 1.27)) (justify left) hide)
     )
-    (property "Manufacturer_Part_Number" "0402WGF1001TCE" (at 176.784 44.196 0)
+    (property "Manufacturer_Part_Number" "0805W8F1801T5E" (at 176.784 44.196 0)
       (effects (font (size 1.27 1.27)) (justify left) hide)
     )
@@
       (effects (font (size 1.27 1.27)) (justify left) hide)
     )
-    (property "Price" "0.0005" (at 188.214 30.226 0)
+    (property "Price" "0.0018" (at 188.214 30.226 0)
       (effects (font (size 1.27 1.27)) hide)
     )
@@
     )
     (property "Extended" "0" (at 188.214 30.226 0)
+      (effects (font (size 1.27 1.27)) hide)
+    )
+    (property "JLC Part Number" "C17398" (at 188.214 30.226 0)
       (effects (font (size 1.27 1.27)) hide)
     )
@@
       (effects (font (size 1.27 1.27)) hide)
     )
+    (property "JLC Part Number" "C1779" (at 222.758 92.202 0)
+      (effects (font (size 1.27 1.27)) hide)
+    )
     (pin "1")
     (pin "2")
@@
     )
     (property "Price" "-" (at 83.058 60.198 0)
+      (effects (font (size 1.27 1.27)) hide)
+    )
+    (property "JLC Part Number" "" (at 83.058 60.198 0)
       (effects (font (size 1.27 1.27)) hide)
     )
@@
       (effects (font (size 1.27 1.27)) hide)
     )
+    (property "JLC Part Number" "C1710" (at 236.728 92.202 0)
+      (effects (font (size 1.27 1.27)) hide)
+    )
     (pin "1")
     (pin "2")
@@
     )
     (property "Price" "-" (at 108.458 60.452 0)
+      (effects (font (size 1.27 1.27)) hide)
+    )
+    (property "JLC Part Number" "" (at 108.458 60.452 0)
       (effects (font (size 1.27 1.27)) hide)
     )
@@
       (effects (font (size 1.27 1.27)) hide)
     )
+    (property "JLC Part Number" "C14663" (at 213.868 92.202 0)
+      (effects (font (size 1.27 1.27)) hide)
+    )
     (pin "1")
     (pin "2")
@@
       (effects (font (size 1.27 1.27)) (justify left) hide)
     )
-    (property "Manufacturer_Part_Number" "0402WGF1001TCE" (at 169.164 42.164 0)
+    (property "Manufacturer_Part_Number" "0805W8F1801T5E" (at 169.164 42.164 0)
       (effects (font (size 1.27 1.27)) (justify left) hide)
     )
@@
       (effects (font (size 1.27 1.27)) (justify left) hide)
     )
-    (property "Price" "0.0005" (at 180.594 28.194 0)
+    (property "Price" "0.0018" (at 180.594 28.194 0)
       (effects (font (size 1.27 1.27)) hide)
     )
@@
       (effects (font (size 1.27 1.27)) hide)
     )
+    (property "JLC Part Number" "C17398" (at 180.594 28.194 0)
+      (effects (font (size 1.27 1.27)) hide)
+    )
