File: EEE3088/Microcontroller_kicad_sch.kicad_sch (KiCad schematic)
At the start: 23 parts, among them J2 Conn_01x24, J3 Conn_01x24

Commit message: C-Branch
Parts:
- removed TP14, TP15, TP17, TP18: TestPoint, TestPoint:TestPoint_Pad_2.0x2.0mm, symbol Connector:TestPoint
Changed lines of the file:
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@@
   (junction (at 203.708 98.552) (diameter 0) (color 0 0 0 0)
   )
-  (junction (at 267.97 33.02) (diameter 0) (color 0 0 0 0)
-  )
   (junction (at 236.728 98.552) (diameter 0) (color 0 0 0 0)
   )
@@
   (junction (at 180.594 57.15) (diameter 0) (color 0 0 0 0)
   )
-  (junction (at 71.12 59.69) (diameter 0) (color 0 0 0 0)
-  )
   (junction (at 236.728 85.852) (diameter 0) (color 0 0 0 0)
   )
   (junction (at 149.86 64.77) (diameter 0) (color 0 0 0 0)
   )
-  (junction (at 171.45 52.07) (diameter 0) (color 0 0 0 0)
-  )
   (junction (at 180.594 38.862) (diameter 0) (color 0 0 0 0)
   )
@@
   )
   (junction (at 213.868 85.852) (diameter 0) (color 0 0 0 0)
-  )
-  (junction (at 72.39 62.23) (diameter 0) (color 0 0 0 0)
   )
   (junction (at 229.87 48.26) (diameter 0) (color 0 0 0 0)
@@
   (no_connect (at 236.22 60.96))
   (no_connect (at 236.22 55.88))
-  (wire (pts (xy 266.7 33.02) (xy 267.97 33.02))
-    (stroke (width 0) (type default))
-  )
   (wire (pts (xy 203.708 85.852) (xy 203.708 88.392))
     (stroke (width 0) (type default))
@@
     (stroke (width 0) (type default))
   )
-  (wire (pts (xy 170.18 52.07) (xy 171.45 52.07))
-    (stroke (width 0) (type default))
-  )
   (wire (pts (xy 219.71 40.64) (xy 219.71 38.735))
     (stroke (width 0) (type default))
@@
     (stroke (width 0) (type default))
   )
-  (wire (pts (xy 267.97 33.02) (xy 270.51 33.02))
+  (wire (pts (xy 266.7 33.02) (xy 270.51 33.02))
     (stroke (width 0) (type default))
   )
@@
     (stroke (width 0) (type default))
   )
-  (wire (pts (xy 72.39 62.23) (xy 74.93 62.23))
+  (wire (pts (xy 68.58 62.23) (xy 74.93 62.23))
     (stroke (width 0) (type default))
   )
@@
     (stroke (width 0) (type default))
   )
-  (wire (pts (xy 68.58 62.23) (xy 72.39 62.23))
-    (stroke (width 0) (type default))
-  )
   (wire (pts (xy 198.12 59.69) (xy 200.66 59.69))
     (stroke (width 0) (type default))
   )
-  (wire (pts (xy 71.12 59.69) (xy 73.66 59.69))
-    (stroke (width 0) (type default))
-  )
-  (wire (pts (xy 68.58 59.69) (xy 71.12 59.69))
+  (wire (pts (xy 68.58 59.69) (xy 73.66 59.69))
     (stroke (width 0) (type default))
   )
@@
     (stroke (width 0) (type default))
   )
-  (wire (pts (xy 171.45 52.07) (xy 176.022 52.07))
+  (wire (pts (xy 170.18 52.07) (xy 176.022 52.07))
     (stroke (width 0) (type default))
   )
@@
     (effects (font (size 1.27 1.27)) (justify right))
   )
-  (symbol (lib_id "Connector:TestPoint") (at 267.97 33.02 0) (unit 1)
-    (in_bom yes) (on_board yes) (dnp no)
-    (property "Reference" "TP15" (at 262.89 26.67 0)
-      (effects (font (size 1.27 1.27)) (justify left))
-    )
-    (property "Value" "TestPoint" (at 259.08 27.94 0)
-      (effects (font (size 1.27 1.27)) (justify left))
-    )
-    (property "Footprint" "TestPoint:TestPoint_Pad_2.0x2.0mm" (at 273.05 33.02 0)
-      (effects (font (size 1.27 1.27)) hide)
-    )
-    (property "Datasheet" "~" (at 273.05 33.02 0)
-      (effects (font (size 1.27 1.27)) hide)
-    )
-    (pin "1")
-    (instances
-      (project "EEE3088"
-        (path "/83bdd5e1-981a-4ca1-9a2f-70dea9f00850/af4ae736-8069-4035-bb69-27168d826fe0"
-          (reference "TP15") (unit 1)
-        )
-      )
-    )
-  )
   (symbol (lib_id "Device:C") (at 246.888 92.202 0) (unit 1)
     (in_bom yes) (on_board yes) (dnp no)
@@
         (path "/83bdd5e1-981a-4ca1-9a2f-70dea9f00850/af4ae736-8069-4035-bb69-27168d826fe0"
           (reference "TP13") (unit 1)
-        )
-      )
-    )
-  )
-  (symbol (lib_id "Connector:TestPoint") (at 72.39 62.23 0) (unit 1)
-    (in_bom yes) (on_board yes) (dnp no) (fields_autoplaced)
-    (property "Reference" "TP18" (at 74.93 58.293 0)
-      (effects (font (size 1.27 1.27)) (justify left))
-    )
-    (property "Value" "TestPoint" (at 74.93 60.833 0)
-      (effects (font (size 1.27 1.27)) (justify left))
-    )
-    (property "Footprint" "TestPoint:TestPoint_Pad_2.0x2.0mm" (at 77.47 62.23 0)
-      (effects (font (size 1.27 1.27)) hide)
-    )
-    (property "Datasheet" "~" (at 77.47 62.23 0)
-      (effects (font (size 1.27 1.27)) hide)
-    )
-    (pin "1")
-    (instances
-      (project "EEE3088"
-        (path "/83bdd5e1-981a-4ca1-9a2f-70dea9f00850/af4ae736-8069-4035-bb69-27168d826fe0"
-          (reference "TP18") (unit 1)
         )
       )
@@
     )
   )
-  (symbol (lib_id "Connector:TestPoint") (at 71.12 59.69 0) (unit 1)
-    (in_bom yes) (on_board yes) (dnp no) (fields_autoplaced)
-    (property "Reference" "TP17" (at 73.66 55.753 0)
-      (effects (font (size 1.27 1.27)) (justify left))
-    )
-    (property "Value" "TestPoint" (at 73.66 58.293 0)
-      (effects (font (size 1.27 1.27)) (justify left))
-    )
-    (property "Footprint" "TestPoint:TestPoint_Pad_2.0x2.0mm" (at 76.2 59.69 0)
-      (effects (font (size 1.27 1.27)) hide)
-    )
-    (property "Datasheet" "~" (at 76.2 59.69 0)
-      (effects (font (size 1.27 1.27)) hide)
-    )
-    (pin "1")
-    (instances
-      (project "EEE3088"
-        (path "/83bdd5e1-981a-4ca1-9a2f-70dea9f00850/af4ae736-8069-4035-bb69-27168d826fe0"
-          (reference "TP17") (unit 1)
-        )
-      )
-    )
-  )
   (symbol (lib_id "power:GND") (at 236.728 98.552 0) (unit 1)
     (in_bom yes) (on_board yes) (dnp no) (fields_autoplaced)
@@
         )
       )
-    )
-  )
-  (symbol (lib_id "Connector:TestPoint") (at 171.45 52.07 0) (unit 1)
-    (in_bom yes) (on_board yes) (dnp no)
-    (property "Reference" "TP14" (at 170.18 45.72 0)
-      (effects (font (size 1.27 1.27)) (justify left))
-    )
-    (property "Value" "TestPoint" (at 166.37 46.99 0)
-      (effects (font (size 1.27 1.27)) (justify left))
-    )
-    (property "Footprint" "TestPoint:TestPoint_Pad_2.0x2.0mm" (at 176.53 52.07 0)
-      (effects (font (size 1.27 1.27)) hide)
-    )
-    (property "Datasheet" "~" (at 176.53 52.07 0)
-      (effects (font (size 1.27 1.27)) hide)
-    )
-    (pin "1")
-    (instances
-      (project "EEE3088"
-        (path "/83bdd5e1-981a-4ca1-9a2f-70dea9f00850/af4ae736-8069-4035-bb69-27168d826fe0"
-          (reference "TP14") (unit 1)
-        )
-      )

Commit message: H_1
Parts:
- removed TP16: TestPoint, TestPoint:TestPoint_Pad_2.0x2.0mm, symbol Connector:TestPoint
Connections:
- net SDASense renamed SDASense_1
Other:
- moved on the sheet: J2, J3

Commit message: Schematic updates
Parts:
- C?: JLC Part Number (none) -> C28323; Manufacturer_Part_Number - -> CL21B105KBFNNNE; Price 0.0087 -> 0.0092
- C? (x2): JLC Part Number C14663 -> C49678; Manufacturer_Part_Number CC0603KRX7R9BB104 -> CC0805KRX7R9BB104; Price 0.01 -> 0.0046
- C?: Price 0.01 -> 0.0112
- C?: Price 0.01 -> 0.0085
- J2, J3: JLC Part Number (none) -> DNP; Manufacturer_Part_Number - -> DNP; Price - -> 0
- J?: Extended 0 -> 1; JLC Part Number (none) -> C404969; Price 0.03 -> 0.0333
- R30, R31: JLC Part Number C17168 -> C17477; Manufacturer_Part_Number 0402WGF0000TCE -> 0805W8F0000T5E; Price 0.0035 -> 0.0022
- R4: Price 0.0018 -> 0.0017
- TP13, TP19, TP20, TP21: Extended (none) -> 0; JLC Part Number (none) -> DNP; Manufacturer_Part_Number (none) -> DNP; Price (none) -> 0
- U?: Price 0.5313 -> 0.4639
- U?: Extended 0 -> 1; Price 0.47 -> 0.4733

Commit message: Schematic + PCB Update
Parts:
- removed J2, J3: Conn_01x24, Connector_PinHeader_1.00mm:PinHeader_1x24_P1.00mm_Vertical, symbol Connector_Generic:Conn_01x24
- removed TP20: TestPoint, TestPoint:TestPoint_Pad_2.0x2.0mm, symbol Connector:TestPoint
- added U6: Header, symbol PCM_UCT:STM32F051C6TG6_Target
- C? (x2): footprint 100n CC0603KRX7R9BB104:CAPC1608X90 -> Capacitor_SMD:C_0805_2012Metric
- C?: footprint 4.7n Cap LIB_0402B472K500NT:CAPC1005X55N -> Capacitor_SMD:C_0805_2012Metric
- C?: footprint 10n Cap CL21B103KBANNNC:CAPC2012X140N -> Capacitor_SMD:C_0805_2012Metric
- R30, R31: footprint Resistor_SMD:R_0402_1005Metric -> Resistor_SMD:R_0805_2012Metric
- R4: footprint 1.8k Ohm Resistor:RESC2013X65N -> Resistor_SMD:R_0805_2012Metric
Connections:
- net +3.3V: now also U6.24 (V+), U6.48 (V+), U6.7 (NRST), U6.9 (V+)
- net EEPROM_SCL: now also U6.32 (PA11)
- net EEPROM_SDA: now also U6.33 (PA12)
- net GND: now also U6.23 (GND), U6.47 (GND), U6.8 (GND)
- net LDR_Vout1: now also U6.11 (PA1)
- net LDR_Vout2: now also U6.12 (PA2)
- net SCLSense: now also U6.21 (PB10)
- net SDASense_1: now also U6.22 (PB11)
- net USB_RXD: now also U6.30 (PA9)
- net USB_TIMIN: now also U6.16 (PA6)
- net USB_TXD: now also U6.31 (PA10)
- net USB_TIMOUT: no longer names the net of U?.8 (XO)
- new net Analogue_Enable1: U6.14 (PA4)
- new net Analogue_Enable2: U6.15 (PA5)
- no-connect marks 5 -> 6
Other:
- note removed: "STM32 PIN 18"
- note removed: "STM32 PIN 19"
- note removed: "STM32 PIN 20"
- note removed: "STM32 PIN 21"
- note removed: "STM32 PIN 23"
- note removed: "STM32 PIN 24"
- note removed: "STM32 PIN 30"
- note removed: "STM32 PIN 31"
- note removed: "STM32 PIN 32"
- note removed: "STM32 PIN 33"
- note removed: "STM32 PIN 45"
- note removed: "STM32 PIN 46"
- note removed: "STM32 PIN 48"
- note removed: "STM32 PIN 8"
- note removed: "STM32 PIN 9"

Commit message: PCB continued again
Parts:
- renumbered R30 to R28, TP13 to TP15, TP21 to TP16, TP19 to TP17, U6 to U5
Changed lines of the file:
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@@
   (symbol (lib_id "power:+3.3V") (at 78.105 38.735 0) (unit 1)
     (in_bom yes) (on_board yes) (dnp no) (fields_autoplaced)
-    (property "Reference" "#PWR049" (at 78.105 42.545 0)
+    (property "Reference" "#PWR035" (at 78.105 42.545 0)
       (effects (font (size 1.27 1.27)) hide)
     )
@@
       (project "EEE3088"
         (path "/83bdd5e1-981a-4ca1-9a2f-70dea9f00850/af4ae736-8069-4035-bb69-27168d826fe0"
-          (reference "#PWR049") (unit 1)
+          (reference "#PWR035") (unit 1)
         )
       )
@@
   (symbol (lib_id "power:+3.3V") (at 98.425 28.575 0) (unit 1)
     (in_bom yes) (on_board yes) (dnp no) (fields_autoplaced)
-    (property "Reference" "#PWR047" (at 98.425 32.385 0)
+    (property "Reference" "#PWR037" (at 98.425 32.385 0)
       (effects (font (size 1.27 1.27)) hide)
     )
@@
       (project "EEE3088"
         (path "/83bdd5e1-981a-4ca1-9a2f-70dea9f00850/af4ae736-8069-4035-bb69-27168d826fe0"
-          (reference "#PWR047") (unit 1)
+          (reference "#PWR037") (unit 1)
         )
       )
@@
   (symbol (lib_id "Connector:TestPoint") (at 198.12 57.15 0) (unit 1)
     (in_bom yes) (on_board yes) (dnp no)
-    (property "Reference" "TP13" (at 196.85 49.53 0)
+    (property "Reference" "TP15" (at 196.85 49.53 0)
       (effects (font (size 1.27 1.27)) (justify left))
     )
@@
       (project "EEE3088"
         (path "/83bdd5e1-981a-4ca1-9a2f-70dea9f00850/af4ae736-8069-4035-bb69-27168d826fe0"
-          (reference "TP13") (unit 1)
+          (reference "TP15") (unit 1)
         )
       )
@@
       (project "EEE3088"
         (path "/83bdd5e1-981a-4ca1-9a2f-70dea9f00850/af4ae736-8069-4035-bb69-27168d826fe0"
-          (reference "#PWR035") (unit 1)
+          (reference "#PWR038") (unit 1)
         )
       )
@@
   (symbol (lib_id "Device:R") (at 24.13 33.02 270) (unit 1)
     (in_bom yes) (on_board yes) (dnp no) (fields_autoplaced)
-    (property "Reference" "R30" (at 24.13 27.94 90)
+    (property "Reference" "R28" (at 24.13 27.94 90)
       (effects (font (size 1.27 1.27)))
     )
@@
       (project "EEE3088"
         (path "/83bdd5e1-981a-4ca1-9a2f-70dea9f00850/af4ae736-8069-4035-bb69-27168d826fe0"
-          (reference "R30") (unit 1)
+          (reference "R28") (unit 1)
         )
       )
@@
       (project "EEE3088"
         (path "/83bdd5e1-981a-4ca1-9a2f-70dea9f00850/af4ae736-8069-4035-bb69-27168d826fe0"
-          (reference "U3") (unit 1)
+          (reference "U6") (unit 1)
         )
       )
@@
   (symbol (lib_id "Connector:TestPoint") (at 229.87 45.72 0) (unit 1)
     (in_bom yes) (on_board yes) (dnp no)
-    (property "Reference" "TP19" (at 232.41 41.783 0)
+    (property "Reference" "TP17" (at 232.41 41.783 0)
       (effects (font (size 1.27 1.27)) (justify left))
     )
@@
       (project "EEE3088"
         (path "/83bdd5e1-981a-4ca1-9a2f-70dea9f00850/af4ae736-8069-4035-bb69-27168d826fe0"
-          (reference "TP19") (unit 1)
+          (reference "TP17") (unit 1)
         )
       )
@@
   (symbol (lib_id "power:GND") (at 97.155 104.775 0) (unit 1)
     (in_bom yes) (on_board yes) (dnp no) (fields_autoplaced)
-    (property "Reference" "#PWR048" (at 97.155 111.125 0)
+    (property "Reference" "#PWR036" (at 97.155 111.125 0)
       (effects (font (size 1.27 1.27)) hide)
     )
@@
       (project "EEE3088"
         (path "/83bdd5e1-981a-4ca1-9a2f-70dea9f00850/af4ae736-8069-4035-bb69-27168d826fe0"
-          (reference "#PWR048") (unit 1)
+          (reference "#PWR036") (unit 1)
         )
       )
@@
       (project "EEE3088"
         (path "/83bdd5e1-981a-4ca1-9a2f-70dea9f00850/af4ae736-8069-4035-bb69-27168d826fe0"
-          (reference "U4") (unit 1)
+          (reference "U7") (unit 1)
         )
       )
@@
       (project "EEE3088"
         (path "/83bdd5e1-981a-4ca1-9a2f-70dea9f00850/af4ae736-8069-4035-bb69-27168d826fe0"
-          (reference "#PWR032") (unit 1)
+          (reference "#PWR034") (unit 1)
         )
       )
@@
       (project "EEE3088"
         (path "/83bdd5e1-981a-4ca1-9a2f-70dea9f00850/af4ae736-8069-4035-bb69-27168d826fe0"
-          (reference "#PWR039") (unit 1)
+          (reference "#PWR042") (unit 1)
         )
       )
@@
   (symbol (lib_id "power:+5V") (at 15.24 33.02 0) (unit 1)
     (in_bom yes) (on_board yes) (dnp no) (fields_autoplaced)
-    (property "Reference" "#PWR046" (at 15.24 36.83 0)
+    (property "Reference" "#PWR033" (at 15.24 36.83 0)
       (effects (font (size 1.27 1.27)) hide)
     )
@@
       (project "EEE3088"
         (path "/83bdd5e1-981a-4ca1-9a2f-70dea9f00850/af4ae736-8069-4035-bb69-27168d826fe0"
-          (reference "#PWR046") (unit 1)
+          (reference "#PWR033") (unit 1)
         )
       )
@@
       (project "EEE3088"
         (path "/83bdd5e1-981a-4ca1-9a2f-70dea9f00850/af4ae736-8069-4035-bb69-27168d826fe0"
-          (reference "#PWR038") (unit 1)
+          (reference "#PWR041") (unit 1)
         )
       )
@@
         )
         (path "/83bdd5e1-981a-4ca1-9a2f-70dea9f00850/af4ae736-8069-4035-bb69-27168d826fe0"
-          (reference "R29") (unit 1)
+          (reference "R30") (unit 1)
         )
       )
@@
   (symbol (lib_id "PCM_UCT:STM32F051C6TG6_Target") (at 97.155 65.405 0) (unit 1)
     (in_bom yes) (on_board yes) (dnp no) (fields_autoplaced)
-    (property "Reference" "U6" (at 102.2859 100.965 0)
+    (property "Reference" "U5" (at 102.2859 100.965 0)
       (effects (font (size 1.27 1.27)) (justify left))
     )
@@
       (project "EEE3088"
         (path "/83bdd5e1-981a-4ca1-9a2f-70dea9f00850/af4ae736-8069-4035-bb69-27168d826fe0"
-          (reference "U6") (unit 1)
+          (reference "U5") (unit 1)
         )
       )
@@
       (project "EEE3088"
         (path "/83bdd5e1-981a-4ca1-9a2f-70dea9f00850/af4ae736-8069-4035-bb69-27168d826fe0"
-          (reference "#PWR036") (unit 1)
+          (reference "#PWR039") (unit 1)
         )
       )
@@
       (project "EEE3088"
         (path "/83bdd5e1-981a-4ca1-9a2f-70dea9f00850/af4ae736-8069-4035-bb69-27168d826fe0"
-          (reference "#PWR037") (unit 1)
+          (reference "#PWR040") (unit 1)
         )
       )
@@
       (project "EEE3088"
         (path "/83bdd5e1-981a-4ca1-9a2f-70dea9f00850/af4ae736-8069-4035-bb69-27168d826fe0"
-          (reference "#PWR044") (unit 1)
+          (reference "#PWR047") (unit 1)
         )
       )
@@
       (project "EEE3088"
         (path "/83bdd5e1-981a-4ca1-9a2f-70dea9f00850/af4ae736-8069-4035-bb69-27168d826fe0"
-          (reference "#PWR040") (unit 1)
+          (reference "#PWR043") (unit 1)
         )
       )
@@
       (project "EEE3088"
         (path "/83bdd5e1-981a-4ca1-9a2f-70dea9f00850/af4ae736-8069-4035-bb69-27168d826fe0"
-          (reference "#PWR042") (unit 1)
+          (reference "#PWR045") (unit 1)
         )
       )
@@
   (symbol (lib_id "Connector:TestPoint") (at 198.12 59.69 180) (unit 1)
     (in_bom yes) (on_board yes) (dnp no) (fields_autoplaced)
-    (property "Reference" "TP21" (at 200.66 62.357 0)
+    (property "Reference" "TP16" (at 200.66 62.357 0)
       (effects (font (size 1.27 1.27)) (justify right))
     )
@@
       (project "EEE3088"
         (path "/83bdd5e1-981a-4ca1-9a2f-70dea9f00850/af4ae736-8069-4035-bb69-27168d826fe0"
-          (reference "TP21") (unit 1)
+          (reference "TP16") (unit 1)
         )
       )
@@
         )
         (path "/83bdd5e1-981a-4ca1-9a2f-70dea9f00850/af4ae736-8069-4035-bb69-27168d826fe0"
-          (reference "R28") (unit 1)
+          (reference "R29") (unit 1)
         )
       )
@@
       (project "EEE3088"
         (path "/83bdd5e1-981a-4ca1-9a2f-70dea9f00850/af4ae736-8069-4035-bb69-27168d826fe0"
-          (reference "#PWR041") (unit 1)
+          (reference "#PWR044") (unit 1)
         )
       )
@@
       (project "EEE3088"
         (path "/83bdd5e1-981a-4ca1-9a2f-70dea9f00850/af4ae736-8069-4035-bb69-27168d826fe0"
-          (reference "#PWR043") (unit 1)
-        )
-      )
+          (reference "#PWR046") (unit 1)
+        )
+      )

Commit message: PCD- stm header added
Parts:
- U5: footprint (none) -> uct_kicad_library:STM32F051C6T6
- U?: footprint AT24C256C-SSHL-T EEPROM Chip:SOIC127P600X175-8N -> Package_SO:SOIC-8-1EP_3.9x4.9mm_P1.27mm_EP2.29x3mm
- U?: footprint CH340G Bridge:SOIC127P600X180-16N -> Package_SO:HTSSOP-16-1EP_4.4x5mm_P0.65mm_EP3.4x5mm
Changed lines of the file:
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@@
       (effects (font (size 1.27 1.27)))
     )
-    (property "Footprint" "AT24C256C-SSHL-T EEPROM Chip:SOIC127P600X175-8N" (at 160.02 59.69 0)
+    (property "Footprint" "Package_SO:SOIC-8-1EP_3.9x4.9mm_P1.27mm_EP2.29x3mm" (at 160.02 59.69 0)
       (effects (font (size 1.27 1.27)) (justify bottom) hide)
     )
@@
       (effects (font (size 1.27 1.27)))
     )
-    (property "Footprint" "CH340G Bridge:SOIC127P600X180-16N" (at 251.46 48.26 0)
+    (property "Footprint" "Package_SO:HTSSOP-16-1EP_4.4x5mm_P0.65mm_EP3.4x5mm" (at 251.46 48.26 0)
       (effects (font (size 1.27 1.27)) (justify bottom) hide)
     )
@@
       (effects (font (size 1.27 1.27)))
     )
-    (property "Footprint" "" (at 97.155 63.5 0)
-      (effects (font (size 1.27 1.27)) hide)
-    )
+    (property "Footprint" "uct_kicad_library:STM32F051C6T6" (at 97.155 63.5 0)
+      (effects (font (size 1.27 1.27)) hide)
+    )

Commit message: PCB-Final
Connections:
- net +3V3 is gone; now on net +3.3V: R31.1, R4.1, R4.1, U?.8 (VCC)
- net LDR_Vout2: now also U5.10 (PA0); no longer U5.12 (PA2)
- net USB_TIMIN: now also U5.45 (PB8); no longer U5.16 (PA6)
- no-connect marks 6 -> 36
Other:
- moved on the sheet: R4, TP15, TP16, U?
