File: EEE3088/Sensing_kicad_sch.kicad_sch (KiCad schematic)
At the start: 28 parts, among them U3 LTR-303ALS-01, U4 LTR-303ALS-01

Commit message: Sense_V1_Submission
Other:
- note added: "Analogue Sensor"
- note added: "Digital Sensor"
- note added: "Secondary Analogue Sensor"
- note added: "Secondary Digital Sensor"
- moved on the sheet: C3, C4, R10, R11, R12, R13, R14, R15, R16, R17, R18, R19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

Commit message: power edit
Parts:
- renumbered R6 to R11, R7 to R12, R22 to R13, R10 to R14, R11 to R15, R8 to R16, R9 to R17, R12 to R18, R13 to R19, R14 to R20, R15 to R21, R16 to R22, R17 to R23, R18 to R24, R19 to R25, R21 to R26, R20 to R27, TP5 to TP10, TP6 to TP11, TP7 to TP12, TP1 to TP6, TP2 to TP7, TP3 to TP8, TP4 to TP9, U3 to U1, U4 to U2

Commit message: updated BOM
Parts:
- C3, C4: footprint CL21B105KBFNNNE -> (none)
Changed lines of the file:
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@@
       (effects (font (size 1.27 1.27)) (justify left))
     )
-    (property "Footprint" "CL21B105KBFNNNE" (at 244.8052 67.31 0)
+    (property "Footprint" "" (at 244.8052 67.31 0)
       (effects (font (size 1.27 1.27)) hide)
     )
@@
       (effects (font (size 1.27 1.27)) (justify left))
     )
-    (property "Footprint" "CL21B105KBFNNNE" (at 247.3452 138.43 0)
-      (effects (font (size 1.27 1.27)) hide)
-    )
+    (property "Footprint" "" (at 247.3452 138.43 0)
+      (effects (font (size 1.27 1.27)) hide)
+    )

Commit message: BOM attempt
Parts:
- C3, C4: Manufacturer_Part_Number (none) -> -
- TP10, TP11, TP12, TP6, TP7, TP8, TP9: Extended (none) -> 0; Manufacturer_Part_Number (none) -> 0; Price (none) -> 0
Changed lines of the file:
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@@
       (effects (font (size 1.27 1.27)) hide)
     )
-    (property "Price" "" (at 179.07 53.34 0)
+    (property "Price" "0" (at 179.07 53.34 0)
       (effects (font (size 1.27 1.27)) hide)
     )
@@
       (effects (font (size 1.27 1.27)) hide)
     )
-    (property "Extended" "" (at 179.07 53.34 0)
+    (property "Extended" "0" (at 179.07 53.34 0)
+      (effects (font (size 1.27 1.27)) hide)
+    )
+    (property "Manufacturer_Part_Number" "0" (at 179.07 53.34 0)
       (effects (font (size 1.27 1.27)) hide)
     )
@@
       (effects (font (size 1.27 1.27)) hide)
     )
-    (property "Price" "" (at 165.1 137.16 0)
+    (property "Price" "0" (at 165.1 137.16 0)
       (effects (font (size 1.27 1.27)) hide)
     )
@@
       (effects (font (size 1.27 1.27)) hide)
     )
-    (property "Extended" "" (at 165.1 137.16 0)
+    (property "Extended" "0" (at 165.1 137.16 0)
+      (effects (font (size 1.27 1.27)) hide)
+    )
+    (property "Manufacturer_Part_Number" "0" (at 165.1 137.16 0)
       (effects (font (size 1.27 1.27)) hide)
     )
@@
       (effects (font (size 1.27 1.27)) hide)
     )
-    (property "Price" "" (at 163.83 58.42 0)
+    (property "Price" "0" (at 163.83 58.42 0)
       (effects (font (size 1.27 1.27)) hide)
     )
@@
       (effects (font (size 1.27 1.27)) hide)
     )
-    (property "Extended" "" (at 163.83 58.42 0)
+    (property "Extended" "0" (at 163.83 58.42 0)
+      (effects (font (size 1.27 1.27)) hide)
+    )
+    (property "Manufacturer_Part_Number" "0" (at 163.83 58.42 0)
       (effects (font (size 1.27 1.27)) hide)
     )
@@
       (effects (font (size 1.27 1.27)) hide)
     )
+    (property "Manufacturer_Part_Number" "-" (at 243.84 63.5 0)
+      (effects (font (size 1.27 1.27)) hide)
+    )
     (pin "1")
     (pin "2")
@@
       (effects (font (size 1.27 1.27)) hide)
     )
-    (property "Price" "" (at 81.28 135.89 0)
+    (property "Price" "0" (at 81.28 135.89 0)
       (effects (font (size 1.27 1.27)) hide)
     )
@@
       (effects (font (size 1.27 1.27)) hide)
     )
-    (property "Extended" "" (at 81.28 135.89 0)
+    (property "Extended" "0" (at 81.28 135.89 0)
+      (effects (font (size 1.27 1.27)) hide)
+    )
+    (property "Manufacturer_Part_Number" "0" (at 81.28 135.89 0)
       (effects (font (size 1.27 1.27)) hide)
     )
@@
       (effects (font (size 1.27 1.27)) hide)
     )
-    (property "Price" "" (at 243.84 57.15 0)
+    (property "Price" "0" (at 243.84 57.15 0)
       (effects (font (size 1.27 1.27)) hide)
     )
@@
       (effects (font (size 1.27 1.27)) hide)
     )
-    (property "Extended" "" (at 243.84 57.15 0)
+    (property "Extended" "0" (at 243.84 57.15 0)
+      (effects (font (size 1.27 1.27)) hide)
+    )
+    (property "Manufacturer_Part_Number" "0" (at 243.84 57.15 0)
       (effects (font (size 1.27 1.27)) hide)
     )
@@
       (effects (font (size 1.27 1.27)) hide)
     )
-    (property "Price" "" (at 77.47 48.26 0)
+    (property "Price" "0" (at 77.47 48.26 0)
       (effects (font (size 1.27 1.27)) hide)
     )
@@
       (effects (font (size 1.27 1.27)) hide)
     )
-    (property "Extended" "" (at 77.47 48.26 0)
+    (property "Extended" "0" (at 77.47 48.26 0)
+      (effects (font (size 1.27 1.27)) hide)
+    )
+    (property "Manufacturer_Part_Number" "0" (at 77.47 48.26 0)
       (effects (font (size 1.27 1.27)) hide)
     )
@@
     )
     (property "Description" "1uF Cap 0805" (at 246.38 134.62 0)
+      (effects (font (size 1.27 1.27)) hide)
+    )
+    (property "Manufacturer_Part_Number" "-" (at 246.38 134.62 0)
       (effects (font (size 1.27 1.27)) hide)
     )
@@
       (effects (font (size 1.27 1.27)) hide)
     )
-    (property "Price" "" (at 176.53 132.08 0)
+    (property "Price" "0" (at 176.53 132.08 0)
       (effects (font (size 1.27 1.27)) hide)
     )
@@
       (effects (font (size 1.27 1.27)) hide)
     )
-    (property "Extended" "" (at 176.53 132.08 0)
-      (effects (font (size 1.27 1.27)) hide)
-    )
+    (property "Extended" "0" (at 176.53 132.08 0)
+      (effects (font (size 1.27 1.27)) hide)
+    )
+    (property "Manufacturer_Part_Number" "0" (at 176.53 132.08 0)
+      (effects (font (size 1.27 1.27)) hide)
+    )

Commit message: BOM_V1_Final
Parts:
- R11, R12, R13, R18, R19, R20, R21: JLC Part Number (none) -> C17168
- R14, R15, R16, R17: JLC Part Number (none) -> C11287
- R22, R23, R24, R25, R26, R27: JLC Part Number (none) -> C17414
- U1, U2: JLC Part Number (none) -> C364577
Changed lines of the file:
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@@
+      (effects (font (size 1.27 1.27)) hide)
+    )
+    (property "JLC Part Number" "C11287" (at 100.33 142.24 0)
       (effects (font (size 1.27 1.27)) hide)
     )
@@
     )
     (property "Manufacturer_Part_Number" "GL3516" (at 101.6 53.34 0)
+      (effects (font (size 1.27 1.27)) hide)
+    )
+    (property "JLC Part Number" "C11287" (at 101.6 53.34 0)
       (effects (font (size 1.27 1.27)) hide)
     )
@@
     )
     (property "Manufacturer_Part_Number" "0402WGF0000TCE" (at 100.33 114.3 0)
+      (effects (font (size 1.27 1.27)) hide)
+    )
+    (property "JLC Part Number" "C17168" (at 100.33 114.3 0)
       (effects (font (size 1.27 1.27)) hide)
     )
@@
       (effects (font (size 1.27 1.27)) hide)
     )
+    (property "JLC Part Number" "C17168" (at 171.45 132.08 0)
+      (effects (font (size 1.27 1.27)) hide)
+    )
     (pin "1")
     (pin "2")
@@
       (effects (font (size 1.27 1.27)) hide)
     )
+    (property "JLC Part Number" "C17168" (at 171.45 137.16 0)
+      (effects (font (size 1.27 1.27)) hide)
+    )
     (pin "1")
     (pin "2")
@@
     )
     (property "Manufacturer_Part_Number" "GL3516" (at 100.33 129.54 0)
+      (effects (font (size 1.27 1.27)) hide)
+    )
+    (property "JLC Part Number" "C11287" (at 100.33 129.54 0)
       (effects (font (size 1.27 1.27)) hide)
     )
@@
       (effects (font (size 1.27 1.27)) hide)
     )
+    (property "JLC Part Number" "" (at 179.07 53.34 0)
+      (effects (font (size 1.27 1.27)) hide)
+    )
     (pin "1")
     (instances
@@
       (effects (font (size 1.27 1.27)) hide)
     )
+    (property "JLC Part Number" "C17414" (at 185.42 40.64 0)
+      (effects (font (size 1.27 1.27)) hide)
+    )
     (pin "1")
     (pin "2")
@@
     )
     (property "Manufacturer_Part_Number" "0805W8F1002T5E" (at 194.31 119.38 0)
+      (effects (font (size 1.27 1.27)) hide)
+    )
+    (property "JLC Part Number" "C17414" (at 194.31 119.38 0)
       (effects (font (size 1.27 1.27)) hide)
     )
@@
     )
     (property "Manufacturer_Part_Number" "LTR-303ALS-01" (at 214.63 55.88 0)
+      (effects (font (size 1.27 1.27)) hide)
+    )
+    (property "JLC Part Number" "C364577" (at 214.63 55.88 0)
       (effects (font (size 1.27 1.27)) hide)
     )
@@
       (effects (font (size 1.27 1.27)) hide)
     )
+    (property "JLC Part Number" "C11287" (at 101.6 40.64 0)
+      (effects (font (size 1.27 1.27)) hide)
+    )
     (pin "1")
     (pin "2")
@@
     )
     (property "Manufacturer_Part_Number" "0805W8F1002T5E" (at 198.12 40.64 0)
+      (effects (font (size 1.27 1.27)) hide)
+    )
+    (property "JLC Part Number" "C17414" (at 198.12 40.64 0)
       (effects (font (size 1.27 1.27)) hide)
     )
@@
       (effects (font (size 1.27 1.27)) hide)
     )
+    (property "JLC Part Number" "" (at 165.1 137.16 0)
+      (effects (font (size 1.27 1.27)) hide)
+    )
     (pin "1")
     (instances
@@
     )
     (property "Manufacturer_Part_Number" "0402WGF0000TCE" (at 63.5 135.89 0)
+      (effects (font (size 1.27 1.27)) hide)
+    )
+    (property "JLC Part Number" "C17168" (at 63.5 135.89 0)
       (effects (font (size 1.27 1.27)) hide)
     )
@@
       (effects (font (size 1.27 1.27)) hide)
     )
+    (property "JLC Part Number" "" (at 163.83 58.42 0)
+      (effects (font (size 1.27 1.27)) hide)
+    )
     (pin "1")
     (instances
@@
       (effects (font (size 1.27 1.27)) hide)
     )
+    (property "JLC Part Number" "" (at 243.84 63.5 0)
+      (effects (font (size 1.27 1.27)) hide)
+    )
     (pin "1")
     (pin "2")
@@
     )
     (property "Description" "Test Point (DNP)" (at 81.28 135.89 0)
+      (effects (font (size 1.27 1.27)) hide)
+    )
+    (property "JLC Part Number" "" (at 81.28 135.89 0)
       (effects (font (size 1.27 1.27)) hide)
     )
@@
       (effects (font (size 1.27 1.27)) hide)
     )
+    (property "JLC Part Number" "C17168" (at 171.45 58.42 0)
+      (effects (font (size 1.27 1.27)) hide)
+    )
     (pin "1")
     (pin "2")
@@
       (effects (font (size 1.27 1.27)) hide)
     )
+    (property "JLC Part Number" "C17414" (at 233.68 41.91 0)
+      (effects (font (size 1.27 1.27)) hide)
+    )
     (pin "1")
     (pin "2")
@@
     )
     (property "Manufacturer_Part_Number" "LTR-303ALS-01" (at 212.09 134.62 0)
+      (effects (font (size 1.27 1.27)) hide)
+    )
+    (property "JLC Part Number" "C364577" (at 212.09 134.62 0)
       (effects (font (size 1.27 1.27)) hide)
     )
@@
       (effects (font (size 1.27 1.27)) hide)
     )
+    (property "JLC Part Number" "" (at 243.84 57.15 0)
+      (effects (font (size 1.27 1.27)) hide)
+    )
     (pin "1")
     (instances
@@
       (effects (font (size 1.27 1.27)) hide)
     )
+    (property "JLC Part Number" "C17168" (at 171.45 53.34 0)
+      (effects (font (size 1.27 1.27)) hide)
+    )
     (pin "1")
     (pin "2")
@@
       (effects (font (size 1.27 1.27)) hide)
     )
+    (property "JLC Part Number" "" (at 77.47 48.26 0)
+      (effects (font (size 1.27 1.27)) hide)
+    )
     (pin "1")
     (instances
@@
       (effects (font (size 1.27 1.27)) hide)
     )
+    (property "JLC Part Number" "C17168" (at 62.23 48.26 0)
+      (effects (font (size 1.27 1.27)) hide)
+    )
     (pin "1")
     (pin "2")
@@
       (effects (font (size 1.27 1.27)) hide)
     )
+    (property "JLC Part Number" "" (at 246.38 134.62 0)
+      (effects (font (size 1.27 1.27)) hide)
+    )
     (pin "1")
     (pin "2")
@@
     )
     (property "Manufacturer_Part_Number" "0805W8F1002T5E" (at 180.34 119.38 0)
+      (effects (font (size 1.27 1.27)) hide)
+    )
+    (property "JLC Part Number" "C17414" (at 180.34 119.38 0)
       (effects (font (size 1.27 1.27)) hide)
     )
@@
       (effects (font (size 1.27 1.27)) hide)
     )
+    (property "JLC Part Number" "" (at 176.53 132.08 0)
+      (effects (font (size 1.27 1.27)) hide)
+    )
     (pin "1")
     (instances
@@
       (effects (font (size 1.27 1.27)) hide)
     )
+    (property "JLC Part Number" "C17414" (at 232.41 119.38 0)
+      (effects (font (size 1.27 1.27)) hide)
+    )

Commit message: Added test points & 0 Ohm
Parts:
- R11, R12, R13, R18, R19, R20, R21: Manufacturer_Name (none) -> ROYALOHM
Changed lines of the file:
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@@
+      (effects (font (size 1.27 1.27)) hide)
+    )
+    (property "Manufacturer_Name" "ROYALOHM" (at 100.33 114.3 0)
       (effects (font (size 1.27 1.27)) hide)
     )
@@
       (effects (font (size 1.27 1.27)) hide)
     )
+    (property "Manufacturer_Name" "ROYALOHM" (at 171.45 132.08 0)
+      (effects (font (size 1.27 1.27)) hide)
+    )
     (pin "1")
     (pin "2")
@@
     )
     (property "JLC Part Number" "C17168" (at 171.45 137.16 0)
+      (effects (font (size 1.27 1.27)) hide)
+    )
+    (property "Manufacturer_Name" "ROYALOHM" (at 171.45 137.16 0)
       (effects (font (size 1.27 1.27)) hide)
     )
@@
       (effects (font (size 1.27 1.27)) hide)
     )
+    (property "Manufacturer_Name" "ROYALOHM" (at 63.5 135.89 0)
+      (effects (font (size 1.27 1.27)) hide)
+    )
     (pin "1")
     (pin "2")
@@
     )
     (property "JLC Part Number" "C17168" (at 171.45 58.42 0)
+      (effects (font (size 1.27 1.27)) hide)
+    )
+    (property "Manufacturer_Name" "ROYALOHM" (at 171.45 58.42 0)
       (effects (font (size 1.27 1.27)) hide)
     )
@@
       (effects (font (size 1.27 1.27)) hide)
     )
+    (property "Manufacturer_Name" "ROYALOHM" (at 171.45 53.34 0)
+      (effects (font (size 1.27 1.27)) hide)
+    )
     (pin "1")
     (pin "2")
@@
       (effects (font (size 1.27 1.27)) hide)
     )
+    (property "Manufacturer_Name" "ROYALOHM" (at 62.23 48.26 0)
+      (effects (font (size 1.27 1.27)) hide)
+    )

Commit message: attempt to assign footprints
Parts:
- R11, R12, R13, R18, R19, R20, R21: footprint 0402WGF0000TCE -> (none)
- R22, R23, R24, R25, R26, R27: footprint 0805W8F1002T5E -> (none)
Changed lines of the file:
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@@
       (effects (font (size 1.27 1.27)) (justify right))
     )
-    (property "Footprint" "0402WGF0000TCE" (at 102.108 114.3 90)
+    (property "Footprint" "" (at 102.108 114.3 90)
       (effects (font (size 1.27 1.27)) hide)
     )
@@
       (effects (font (size 1.27 1.27)))
     )
-    (property "Footprint" "0402WGF0000TCE" (at 171.45 130.302 90)
+    (property "Footprint" "" (at 171.45 130.302 90)
       (effects (font (size 1.27 1.27)) hide)
     )
@@
       (effects (font (size 1.27 1.27)))
     )
-    (property "Footprint" "0402WGF0000TCE" (at 171.45 138.938 90)
+    (property "Footprint" "" (at 171.45 138.938 90)
       (effects (font (size 1.27 1.27)) hide)
     )
@@
       (effects (font (size 1.27 1.27)) (justify left))
     )
-    (property "Footprint" "0805W8F1002T5E" (at 183.642 40.64 90)
+    (property "Footprint" "" (at 183.642 40.64 90)
       (effects (font (size 1.27 1.27)) hide)
     )
@@
       (effects (font (size 1.27 1.27)) (justify left))
     )
-    (property "Footprint" "0805W8F1002T5E" (at 192.532 119.38 90)
+    (property "Footprint" "" (at 192.532 119.38 90)
       (effects (font (size 1.27 1.27)) hide)
     )
@@
       (effects (font (size 1.27 1.27)) (justify left))
     )
-    (property "Footprint" "0805W8F1002T5E" (at 196.342 40.64 90)
+    (property "Footprint" "" (at 196.342 40.64 90)
       (effects (font (size 1.27 1.27)) hide)
     )
@@
       (effects (font (size 1.27 1.27)))
     )
-    (property "Footprint" "0402WGF0000TCE" (at 63.5 137.668 90)
+    (property "Footprint" "" (at 63.5 137.668 90)
       (effects (font (size 1.27 1.27)) hide)
     )
@@
       (effects (font (size 1.27 1.27)))
     )
-    (property "Footprint" "0402WGF0000TCE" (at 171.45 60.198 90)
+    (property "Footprint" "" (at 171.45 60.198 90)
       (effects (font (size 1.27 1.27)) hide)
     )
@@
       (effects (font (size 1.27 1.27)) (justify left))
     )
-    (property "Footprint" "0805W8F1002T5E" (at 231.902 41.91 90)
+    (property "Footprint" "" (at 231.902 41.91 90)
       (effects (font (size 1.27 1.27)) hide)
     )
@@
       (effects (font (size 1.27 1.27)))
     )
-    (property "Footprint" "0402WGF0000TCE" (at 171.45 55.118 90)
+    (property "Footprint" "" (at 171.45 55.118 90)
       (effects (font (size 1.27 1.27)) hide)
     )
@@
       (effects (font (size 1.27 1.27)))
     )
-    (property "Footprint" "0402WGF0000TCE" (at 62.23 46.482 90)
+    (property "Footprint" "" (at 62.23 46.482 90)
       (effects (font (size 1.27 1.27)) hide)
     )
@@
       (effects (font (size 1.27 1.27)) (justify left))
     )
-    (property "Footprint" "0805W8F1002T5E" (at 178.562 119.38 90)
+    (property "Footprint" "" (at 178.562 119.38 90)
       (effects (font (size 1.27 1.27)) hide)
     )
@@
       (effects (font (size 1.27 1.27)) (justify left))
     )
-    (property "Footprint" "0805W8F1002T5E" (at 230.632 119.38 90)
-      (effects (font (size 1.27 1.27)) hide)
-    )
+    (property "Footprint" "" (at 230.632 119.38 90)
+      (effects (font (size 1.27 1.27)) hide)
+    )
