File: EEE3088/EEE3088.kicad_sch (KiCad schematic)
At the start: 0 parts

Commit message: Schematic updates
Other:
- sheet Sensing_Subsystem ports: added Analogue_Enable_1, Analogue_Enable_2; removed none
Changed lines of the file:
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@@
+      (effects (font (size 1.27 1.27)) (justify left))
+    )
+    (pin "Analogue_Enable_1" input (at 200.66 96.52 180)
+      (effects (font (size 1.27 1.27)) (justify left))
+    )
+    (pin "Analogue_Enable_2" input (at 200.66 99.06 180)
       (effects (font (size 1.27 1.27)) (justify left))
     )

Commit message: Schematic + PCB Update
Other:
- sheet Microcontroller ports: added Analogue_Enable1, Analogue_Enable2; removed none
Changed lines of the file:
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@@
+    (stroke (width 0) (type default))
+  )
+  (wire (pts (xy 170.18 99.06) (xy 200.66 99.06))
     (stroke (width 0) (type default))
   )
   (wire (pts (xy 170.18 93.98) (xy 200.66 93.98))
+    (stroke (width 0) (type default))
+  )
+  (wire (pts (xy 170.18 96.52) (xy 200.66 96.52))
     (stroke (width 0) (type default))
   )
@@
       (effects (font (size 1.27 1.27)) (justify right))
     )
+    (pin "Analogue_Enable1" input (at 170.18 96.52 0)
+      (effects (font (size 1.27 1.27)) (justify right))
+    )
+    (pin "Analogue_Enable2" input (at 170.18 99.06 0)
+      (effects (font (size 1.27 1.27)) (justify right))
+    )
