File: EEE3088/EEE3088.kicad_pcb (KiCad board)
At the start: 2 copper layers, 100 x 100 mm, 74 parts, among them J1 MICROXNJ, J2 Conn_01x24, J3 Conn_01x24, U1 LTR-303ALS-01, U2 LTR-303ALS-01, U3 AT24C256C-SSHL-T, U4 CH340G

Commit message: H_1
Parts:
- moved Battery-Charger1 299.2 mm to (-171.2, 63.0)
- moved C1 299.2 mm to (-174.5, 68.1)
- moved C2 299.2 mm to (-171.2, 68.1)
- moved C3 299.2 mm to (-206.2, 67.0)
- moved C4 299.2 mm to (-112.6, 68.1)
- moved C5 299.2 mm to (-146.8, 44.7)
- moved C6 299.2 mm to (-149.4, 44.7)
- moved C9 299.2 mm to (-151.9, 44.7)
- moved J1 299.2 mm to (-145.0, 12.0)
- moved J2 299.2 mm to (-144.5, 40.1)
- moved J3 299.2 mm to (-144.3, 50.3)
- moved LED1 299.2 mm to (-155.9, 60.4)
- moved LED2 299.2 mm to (-155.9, 65.5)
- moved Op-Amp1 299.2 mm to (-128.5, 81.8)
- moved P-Mos1 299.2 mm to (-118.0, 86.8)
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Routing:
- removed copper zone on B.Cu, net GND

Commit message: Schematic + PCB Update
Parts:
- removed J2, J3: Conn_01x24, Connector_PinHeader_1.00mm:PinHeader_1x24_P1.00mm_Vertical
- removed TP16, TP20: TestPoint, TestPoint:TestPoint_Pad_2.0x2.0mm
- added Q1: MMDT2222A, Package_TO_SOT_SMD:SOT-363_SC-70-6, F.Cu at (100.1, 87.5)
- added TP12: TestPoint, TestPoint:TestPoint_Pad_2.0x2.0mm, F.Cu at (-87.0, 184.3)
- added TP14: TestPoint, TestPoint:TestPoint_Pad_2.0x2.0mm, F.Cu at (-79.5, 185.2)
- C1, C2: footprint CL10A106KP8NNNC:CAPC1608X90N -> Capacitor_SMD:C_0805_2012Metric
- C5, C6: footprint 100n CC0603KRX7R9BB104:CAPC1608X90 -> Capacitor_SMD:C_0805_2012Metric
- C7: footprint 4.7n Cap LIB_0402B472K500NT:CAPC1005X55N -> Capacitor_SMD:C_0805_2012Metric
- C8: footprint 10n Cap CL21B103KBANNNC:CAPC2012X140N -> Capacitor_SMD:C_0805_2012Metric
- R10, R11, R12, R13, R18, R19, R20, R21, R30, R31, R4, R6, R8, R9: footprint Resistor_SMD:R_0402_1005Metric -> Resistor_SMD:R_0805_2012Metric
- R2, R32, R5: footprint My1.2k:RESC1608X55N -> Resistor_SMD:R_0805_2012Metric
- R28, R29: footprint 1.8k Ohm Resistor:RESC2013X65N -> Resistor_SMD:R_0805_2012Metric
- R3: footprint My100k:RESC3116X65N -> Resistor_SMD:R_0805_2012Metric
- R7: footprint My1M:RESC2013X65N -> Resistor_SMD:R_0805_2012Metric
- moved R2 294.9 mm to (109.5, 135.8), turned to 180 degrees
- moved C1 291.5 mm to (109.6, 133.5)
- moved Battery-Charger1 283.6 mm to (103.0, 135.3), turned to 180 degrees
- moved C2 274.5 mm to (95.9, 131.4)
- moved TP2 274.5 mm to (101.4, 129.5), turned to -90 degrees
- moved R6 272.1 mm to (95.9, 129.2)
- moved R32 271.9 mm to (95.9, 135.9), turned to 180 degrees
- moved R11 270.9 mm to (143.8, 70.0), turned to -90 degrees
- moved TP6 269.5 mm to (143.8, 65.8)
- moved R5 267.5 mm to (95.9, 133.7), turned to 0 degrees
- moved R13 263.7 mm to (59.7, 69.4), turned to -90 degrees
- moved R14 263.6 mm to (55.9, 53.9)
- moved TP9 263.2 mm to (141.6, 92.1)
- moved R15 263.1 mm to (56.4, 138.7)
- moved C4 263.0 mm to (147.7, 105.6)
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Connections:
- net /Microcontroller/SDASense renamed /Microcontroller/SDASense_1
- Op-Amp1 pad 5: GND -> unconnected-(Op-Amp1-VINB+-Pad5)
- Op-Amp1 pad 6: GND -> unconnected-(Op-Amp1-VINB--Pad6)
- R13 pad 2: +3.3V -> Net-(Q1A-E1)
- R16 pad 1: +3.3V -> Net-(Q1B-E2)
- TP5 pad 1: Net-(Voltage-Regulator-2-VO) -> +3.3V
- U4 pad 8: /Microcontroller/USB_TIMOUT -> unconnected-(U4-XO-Pad8)
Routing:
- net +3.3V: track 295.7 -> 72.1 mm, vias 4 -> 2
- net /Microcontroller/SCLSense: track 112.8 -> 2.66 mm, vias 1 -> 0
- net +5V: track 103.2 -> 0.13 mm, vias 3 -> 0
- net /Microcontroller/SDASense_1: track 106.8 -> 34.5 mm, vias 2 -> 0
- net /Power_Subsystem/Vbat: track 29.0 -> 0.00 mm
- net GND: track 119.2 -> 96.8 mm, vias 7 -> 4
- net unconnected-(U4-XO-Pad8): track 0.00 -> 21.2 mm
- net /Microcontroller/USB_TIMOUT: track 21.2 -> 0.00 mm
- net Net-(Battery-Holder1-PadP): track 26.1 -> 5.45 mm
- net /Microcontroller/LDR_Vout1: track 66.0 -> 46.7 mm, vias 1 -> 0
- net /Microcontroller/LDR_Vout2: track 51.8 -> 34.0 mm, vias 2 -> 0
- net Net-(Battery-Charger1-BAT): track 13.1 -> 0.09 mm
- net Net-(R13-Pad1): track 6.21 -> 16.3 mm
- net Net-(Voltage-Regulator-2-VO): track 9.38 -> 0.00 mm
- net Net-(LED1-Pad1): track 7.81 -> 0.00 mm
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Other:
- outline, holes or cut-outs redrawn

Commit message: PCB continued again
Parts:
- removed Battery-Charger1: TP4056, TP4056:SOP127P600X175-9N
- removed Op-Amp1: MCP6002T-I_SN, Myopamp:SOIC127P600X175-8N
- removed R32: 1k, Resistor_SMD:R_0805_2012Metric
- removed TP19, TP21, TP22: TestPoint, TestPoint:TestPoint_Pad_2.0x2.0mm
- removed Voltage-Regulator-1, Voltage-Regulator-2: HT7533-1, HT7533-1:SOT89
- added R1: 1k, Resistor_SMD:R_0805_2012Metric, F.Cu at (118.2, 181.6)
- added TP15: TestPoint, TestPoint:TestPoint_Pad_2.0x2.0mm, F.Cu at (112.0, 182.1)
- added TP16: TestPoint, TestPoint:TestPoint_Pad_2.0x2.0mm, F.Cu at (112.0, 186.2)
- added TP17: TestPoint, TestPoint:TestPoint_Pad_2.0x2.0mm, F.Cu at (112.0, 190.2)
- R2: value 1.2k -> 100k
- R28: value 1.8k -> 0
- R3: value 100k -> 1.2k
- R30: value 0 -> 1.8k
- R7: value 1M -> 0
- R8: value 0 -> 1M
- U3: value AT24C256C-SSHL-T -> LTR-303ALS-01; footprint AT24C256C-SSHL-T EEPROM Chip:SOIC127P600X175-8N -> OptoDevice:Lite-On_LTR-303ALS-01
- U4: value CH340G -> LTR-303ALS-01; footprint CH340G Bridge:SOIC127P600X180-16N -> OptoDevice:Lite-On_LTR-303ALS-01
- moved TP12 246.5 mm to (141.6, 91.9)
- moved R9 225.4 mm to (87.9, 179.6), turned to -90 degrees
- moved TP3 224.2 mm to (108.7, 168.8)
- moved TP4 223.7 mm to (98.4, 179.8)
- moved R8 218.7 mm to (98.8, 175.5)
- moved TP5 216.5 mm to (83.6, 179.8)
- moved TP1 209.9 mm to (128.1, 175.9)
- moved P-Mos1 209.0 mm to (128.8, 171.7), turned to 0 degrees
- moved R7 208.8 mm to (98.8, 172.8), turned to 180 degrees
- moved Z1 207.3 mm to (124.0, 173.2), turned to 180 degrees
- moved N-Mos1 206.1 mm to (103.7, 174.3)
- moved R4 203.4 mm to (124.1, 175.9), turned to 180 degrees
- moved R3 201.5 mm to (123.9, 170.3), turned to 0 degrees
- moved R10 195.9 mm to (93.7, 179.7), turned to -90 degrees
- moved TP14 187.1 mm to (87.5, 100.7)
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Connections:
- C2 pad 1: Net-(Battery-Charger1-BAT) -> Net-(U8-BAT)
- N-Mos1 pad 1: Net-(Op-Amp1-VOUTA) -> Net-(U9-VOUTA)
- R10 pad 1: Net-(Voltage-Regulator-1-VO) -> Net-(U1-VO)
- R18 pad 2: Net-(U2-SDA) -> Net-(U4-SDA)
- R19 pad 2: Net-(U2-SCL) -> Net-(U4-SCL)
- R2 pad 2: Net-(Battery-Charger1-PROG) -> Net-(Z1-A)
- R20 pad 1: Net-(U1-SDA) -> Net-(U3-SDA)
- R21 pad 2: Net-(U1-SCL) -> Net-(U3-SCL)
- R22 pad 2: Net-(U1-SCL) -> Net-(U3-SCL)
- R23 pad 2: Net-(U2-SCL) -> Net-(U4-SCL)
- R24 pad 2: Net-(U1-SDA) -> Net-(U3-SDA)
- R25 pad 2: Net-(U2-SDA) -> Net-(U4-SDA)
- R26 pad 2: Net-(U1-INT) -> Net-(U3-INT)
- R27 pad 2: Net-(U2-INT) -> Net-(U4-INT)
- R28 pad 1: +3V3 -> Net-(J1-VBUS)
- R28 pad 2: /Microcontroller/EEPROM_SCL -> +5V
- R29 pad 2: /Microcontroller/EEPROM_SDA -> /Microcontroller/EEPROM_SCL
- R3 pad 2: Net-(Z1-A) -> Net-(U8-PROG)
- R30 pad 1: Net-(J1-VBUS) -> +3V3
- R30 pad 2: +5V -> /Microcontroller/EEPROM_SDA
- R31 pad 2: Net-(U4-V3) -> Net-(U7-V3)
- R6 pad 1: Net-(Battery-Charger1-BAT) -> Net-(U8-BAT)
- R7 pad 2: GND -> /Power_Subsystem/V-Reg
- R8 pad 2: /Power_Subsystem/V-Reg -> GND
- TP10 pad 1: Net-(U1-SDA) -> Net-(R12-Pad2)
- TP11 pad 1: Net-(U2-SDA) -> Net-(U3-SDA)
- TP12 pad 1: GND -> Net-(U3-SCL)
- TP13 pad 1: /Microcontroller/EEPROM_SCL -> Net-(U4-SDA)
- TP14 pad 1: +5V -> Net-(U4-SCL)
- TP2 pad 1: Net-(Battery-Charger1-BAT) -> GND
- TP3 pad 1: Net-(N-Mos1-Pad2) -> +5V
- TP4 pad 1: Net-(Voltage-Regulator-1-VO) -> Net-(U8-BAT)
- TP5 pad 1: +3.3V -> Net-(U9-VOUTA)
- TP6 pad 1: Net-(R11-Pad1) -> Net-(N-Mos1-Pad2)
- TP7 pad 1: Net-(R12-Pad2) -> Net-(U1-VO)
- TP8 pad 1: Net-(U2-SCL) -> +3.3V
- TP9 pad 1: Net-(U1-SCL) -> Net-(R11-Pad1)
- U3 pad 1: GND -> +3.3V
- U3 pad 2: GND -> unconnected-(U3-NC-Pad2)
- U3 pad 4: GND -> Net-(U3-SCL)
- U3 pad 5: /Microcontroller/EEPROM_SDA -> Net-(U3-INT)
- U3 pad 6: /Microcontroller/EEPROM_SCL -> Net-(U3-SDA)
- U4 pad 1: GND -> +3.3V
- U4 pad 2: /Microcontroller/USB_TXD -> unconnected-(U4-NC-Pad2)
- U4 pad 3: /Microcontroller/USB_RXD -> GND
- U4 pad 4: Net-(U4-V3) -> Net-(U4-SCL)
- U4 pad 5: /Microcontroller/USB_D+ -> Net-(U4-INT)
- U4 pad 6: /Microcontroller/USB_D- -> Net-(U4-SDA)
Routing:
- net (no net): track 0.00 -> 62.2 mm, vias 0 -> 4
- net /Power_Subsystem/V-pos: track 49.8 -> 0.00 mm
- net /Microcontroller/EEPROM_SDA: track 28.0 -> 0.00 mm
- net /Microcontroller/EEPROM_SCL: track 28.4 -> 56.4 mm
- net Net-(Voltage-Regulator-1-VO): track 23.1 -> 0.00 mm
- net unconnected-(U4-XO-Pad8): track 21.2 -> 0.00 mm
- net Net-(N-Mos1-Pad2): track 17.1 -> 0.00 mm
- net Net-(Z1-K): track 16.1 -> 0.00 mm
- net /Microcontroller/USB_RXD: track 15.6 -> 0.00 mm, vias 1 -> 0
- net /Microcontroller/USB_TXD: track 12.9 -> 0.00 mm, vias 1 -> 0
- net Net-(U4-V3): track 12.5 -> 0.00 mm, vias 2 -> 0
- net /Power_Subsystem/3.3-back: track 11.5 -> 0.00 mm
- net Net-(Z1-A): track 11.2 -> 0.00 mm
- net Net-(Op-Amp1-VOUTA): track 9.31 -> 0.00 mm
- net GND: track 96.8 -> 90.5 mm, vias 4 -> 2
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Other:
- board text removed: "Reverse Polarity Protection"

Commit message: PCD- stm header added
Parts:
- added U5: Header, uct_kicad_library:STM32F051C6T6, F.Cu at (99.6, 101.3)
- added U6: AT24C256C-SSHL-T, Package_SO:SOIC-8-1EP_3.9x4.9mm_P1.27mm_EP2.29x3mm, F.Cu at (-135.6, 24.6)
- added U7: CH340G, Package_SO:HTSSOP-16-1EP_4.4x5mm_P0.65mm_EP3.4x5mm, F.Cu at (65.3, 181.7)
- added U8: TP4056, Package_SO:SOP-8-1EP_4.57x4.57mm_P1.27mm_EP4.57x4.45mm, F.Cu at (67.6, 173.2)
- added U9: MCP6002T-I_SN, Package_SO:SOIC-8-1EP_3.9x4.9mm_P1.27mm_EP2.29x3mm, F.Cu at (86.5, 186.9)
- U1, U2: value LTR-303ALS-01 -> HT7533-1; footprint OptoDevice:Lite-On_LTR-303ALS-01 -> Package_TO_SOT_SMD:SOT-89-3
- moved U3 318.9 mm to (147.1, 100.2), turned to 180 degrees
- moved TP13 225.0 mm to (57.0, 90.8)
- moved U4 211.8 mm to (52.5, 99.6), turned to 0 degrees
- moved U1 84.9 mm to (94.3, 166.7), turned to 90 degrees
- moved U2 82.4 mm to (100.4, 166.7), turned to 90 degrees
- moved TP14 31.9 mm to (56.9, 109.7)
- moved Battery-Holder1 22.6 mm to (101.0, 122.6)
- moved TP11 17.1 mm to (142.1, 108.7)
- moved TP12 0.38 mm to (142.0, 91.9)
Connections:
- U1 pad 1: +3.3V -> GND
- U1 pad 2: unconnected-(U1-NC-Pad2) -> /Power_Subsystem/V-Reg
- U1 pad 3: GND -> Net-(U1-VO)
- U2 pad 1: +3.3V -> GND
- U2 pad 2: unconnected-(U2-NC-Pad2) -> /Power_Subsystem/V-Reg
- U2 pad 3: GND -> Net-(U2-VO)
Routing:
- net /Microcontroller/EEPROM_SCL: track 56.4 -> 28.0 mm
- net +5V: track 0.04 -> 28.4 mm
- net (no net): track 62.2 -> 49.7 mm, vias 4 -> 2
- net Net-(U7-V3): track 0.00 -> 12.5 mm, vias 0 -> 2
- net Net-(U4-SCL): track 0.00 -> 12.1 mm
- net Net-(U2-SCL): track 12.1 -> 0.00 mm
- net Net-(U3-SDA): track 0.00 -> 10.7 mm
- net Net-(U1-SDA): track 10.7 -> 0.00 mm
- net Net-(U3-SCL): track 0.00 -> 10.4 mm
- net Net-(U1-SCL): track 10.4 -> 0.00 mm
- net Net-(U4-SDA): track 0.00 -> 10.3 mm
- net Net-(U2-SDA): track 10.3 -> 0.00 mm
- net Net-(U3-INT): track 0.00 -> 3.42 mm
- net Net-(U1-INT): track 3.42 -> 0.00 mm
- net Net-(U4-INT): track 0.00 -> 3.02 mm
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