File: KiCAD_Project/Power_kicad_sch.kicad_sch (KiCad schematic)
At the start: 30 parts, among them P1 AO3401A, U1 HT7533-1, U1 TP4056, U2 HT7533-1, U9 MCP6002T-I_SN

Commit message: unimportant
Other:
- note added: "Note: Low Voltage Lockout may draw power when device is off."
Changed lines of the file:
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@@
+    (effects (font (size 1.27 1.27)) (justify left bottom))
+  )
+  (text "Note: Low Voltage Lockout may draw power when device is off."
+    (at 104.775 107.315 0)
     (effects (font (size 1.27 1.27)) (justify left bottom))
   )
@@
       (effects (font (size 1.27 1.27)) hide)
     )
+    (pin "1")
     (pin "2")
-    (pin "1")
     (instances
       (project "Power_kicad_sch"
